File: HARDWARE/BMS_LV_2022/Balance.sch (KiCad schematic (older format))
At the start: 9 parts, among them Q2 Q_NMOS_GSD

Commit message: Some footprint changes
Parts:
- D7: footprint Diode_SMD:D_SMB -> Diode_SMD:D_SOD-110
Changed lines of the file:
@@
 $Descr A4 11693 8268
 encoding utf-8
-Sheet 8 13
+Sheet 7 13
 Title "Balance part of LTC6810"
 Date ""
@@
 AR Path="/61996AA1/61A3B341/6199E2E8" Ref="R41"  Part="1"
 AR Path="/61996AA1/61A3CF51/6199E2E8" Ref="R46"  Part="1"
-F 0 "R46" H 5592 4004 50  0000 R CNN
+F 0 "R41" H 5592 4004 50  0000 R CNN
 F 1 "30" H 5592 4095 50  0000 R CNN
 F 2 "Resistor_SMD:R_2512_6332Metric" H 5650 4050 50  0001 C CNN
@@
 AR Path="/61996AA1/61A3B341/6199F863" Ref="R42"  Part="1"
 AR Path="/61996AA1/61A3CF51/6199F863" Ref="R47"  Part="1"
-F 0 "R47" H 6042 4004 50  0000 R CNN
+F 0 "R42" H 6042 4004 50  0000 R CNN
 F 1 "30" H 6042 4095 50  0000 R CNN
 F 2 "Resistor_SMD:R_2512_6332Metric" H 6100 4050 50  0001 C CNN
@@
 AR Path="/61996AA1/61A3B341/619A21A9" Ref="R43"  Part="1"
 AR Path="/61996AA1/61A3CF51/619A21A9" Ref="R48"  Part="1"
-F 0 "R48" V 6254 3850 50  0000 C CNN
+F 0 "R43" V 6254 3850 50  0000 C CNN
 F 1 "330" V 6345 3850 50  0000 C CNN
 F 2 "Resistor_SMD:R_0603_1608Metric" H 6450 3850 50  0001 C CNN
@@
 AR Path="/61996AA1/61A3B341/619A6565" Ref="D14"  Part="1"
 AR Path="/61996AA1/61A3CF51/619A6565" Ref="D16"  Part="1"
-F 0 "D16" H 6450 4535 50  0000 C CNN
+F 0 "D14" H 6450 4535 50  0000 C CNN
 F 1 "LED_RED" H 6450 4444 50  0000 C CNN
 F 2 "LED_SMD:LED_0603_1608Metric" V 6450 4300 50  0001 C CNN
@@
 AR Path="/61996AA1/61A3B341/619B0D16" Ref="R44"  Part="1"
 AR Path="/61996AA1/61A3CF51/619B0D16" Ref="R49"  Part="1"
-F 0 "R49" V 6254 4950 50  0000 C CNN
+F 0 "R44" V 6254 4950 50  0000 C CNN
 F 1 "1k" V 6345 4950 50  0000 C CNN
 F 2 "Resistor_SMD:R_0603_1608Metric" H 6450 4950 50  0001 C CNN
@@
 AR Path="/61996AA1/61A3B341/619B293B" Ref="D15"  Part="1"
 AR Path="/61996AA1/61A3CF51/619B293B" Ref="D17"  Part="1"
-F 0 "D17" H 6450 5043 50  0000 C CNN
+F 0 "D15" H 6450 5043 50  0000 C CNN
 F 1 "D_Zener 9.1V" H 6450 5134 50  0000 C CNN
-F 2 "Diode_SMD:D_SMB" V 6450 5250 50  0001 C CNN
+F 2 "Diode_SMD:D_SOD-110" V 6450 5250 50  0001 C CNN
 F 3 "~" V 6450 5250 50  0001 C CNN
 	1    6450 5250
@@
 AR Path="/61996AA1/61A3B341/619B7EAD" Ref="R45"  Part="1"
 AR Path="/61996AA1/61A3CF51/619B7EAD" Ref="R50"  Part="1"
-F 0 "R50" V 6754 3600 50  0000 C CNN
+F 0 "R45" V 6754 3600 50  0000 C CNN
 F 1 "100" V 6845 3600 50  0000 C CNN
 F 2 "Resistor_SMD:R_0603_1608Metric" H 6950 3600 50  0001 C CNN
@@
 AR Path="/61996AA1/61A3B341/619BEE0A" Ref="C23"  Part="1"
 AR Path="/61996AA1/61A3CF51/619BEE0A" Ref="C24"  Part="1"
-F 0 "C24" H 7242 3846 50  0000 L CNN
+F 0 "C23" H 7242 3846 50  0000 L CNN
 F 1 "10nF" H 7242 3755 50  0000 L CNN
 F 2 "Capacitor_SMD:C_0603_1608Metric" H 7150 3800 50  0001 C CNN
@@
 AR Path="/61996AA1/61A3B341/619C00A1" Ref="#PWR036"  Part="1"
 AR Path="/61996AA1/61A3CF51/619C00A1" Ref="#PWR037"  Part="1"
-F 0 "#PWR037" H 7150 3700 50  0001 C CNN
+F 0 "#PWR036" H 7150 3700 50  0001 C CNN
 F 1 "GND" H 7155 3777 50  0000 C CNN
 F 2 "" H 7150 3950 50  0001 C CNN
@@
 AR Path="/61996AA1/61A3B341/619A7C3D" Ref="Q6"  Part="1"
 AR Path="/61996AA1/61A3CF51/619A7C3D" Ref="Q7"  Part="1"
-F 0 "Q7" H 6405 4604 50  0000 L CNN
+F 0 "Q6" H 6405 4604 50  0000 L CNN
 F 1 "Q_NMOS_GSD" H 6405 4695 50  0000 L CNN
 F 2 "Package_TO_SOT_SMD:SOT-23" H 6400 4750 50  0001 C CNN
