File: HARDWARE/BMS_LV_2022/Balance.sch (KiCad schematic (older format))
At the start: 9 parts

Commit message: Electrical Rules Checker fixes
Parts:
- gave numbers to parts that had none: 9
Changed lines of the file:
@@
 	2950 1950 3200 1950
 $Comp
-L Device:R_Small R?
+L Device:R_Small R21
 U 1 1 6199E2E8
 P 2500 2150
-AR Path="/61996AA1/6199D637/6199E2E8" Ref="R?"  Part="1"
-AR Path="/61996AA1/61A346F1/6199E2E8" Ref="R?"  Part="1"
-AR Path="/61996AA1/61A395F7/6199E2E8" Ref="R?"  Part="1"
-AR Path="/61996AA1/61A3A424/6199E2E8" Ref="R?"  Part="1"
-AR Path="/61996AA1/61A3B341/6199E2E8" Ref="R?"  Part="1"
-AR Path="/61996AA1/61A3CF51/6199E2E8" Ref="R?"  Part="1"
-F 0 "R?" H 2442 2104 50  0000 R CNN
+AR Path="/61996AA1/6199D637/6199E2E8" Ref="R21"  Part="1"
+AR Path="/61996AA1/61A346F1/6199E2E8" Ref="R26"  Part="1"
+AR Path="/61996AA1/61A395F7/6199E2E8" Ref="R31"  Part="1"
+AR Path="/61996AA1/61A3A424/6199E2E8" Ref="R36"  Part="1"
+AR Path="/61996AA1/61A3B341/6199E2E8" Ref="R41"  Part="1"
+AR Path="/61996AA1/61A3CF51/6199E2E8" Ref="R46"  Part="1"
+F 0 "R46" H 2442 2104 50  0000 R CNN
 F 1 "30" H 2442 2195 50  0000 R CNN
 F 2 "" H 2500 2150 50  0001 C CNN
@@
 $EndComp
 $Comp
-L Device:R_Small R?
+L Device:R_Small R22
 U 1 1 6199F863
 P 2950 2150
-AR Path="/61996AA1/6199D637/6199F863" Ref="R?"  Part="1"
-AR Path="/61996AA1/61A346F1/6199F863" Ref="R?"  Part="1"
-AR Path="/61996AA1/61A395F7/6199F863" Ref="R?"  Part="1"
-AR Path="/61996AA1/61A3A424/6199F863" Ref="R?"  Part="1"
-AR Path="/61996AA1/61A3B341/6199F863" Ref="R?"  Part="1"
-AR Path="/61996AA1/61A3CF51/6199F863" Ref="R?"  Part="1"
-F 0 "R?" H 2892 2104 50  0000 R CNN
+AR Path="/61996AA1/6199D637/6199F863" Ref="R22"  Part="1"
+AR Path="/61996AA1/61A346F1/6199F863" Ref="R27"  Part="1"
+AR Path="/61996AA1/61A395F7/6199F863" Ref="R32"  Part="1"
+AR Path="/61996AA1/61A3A424/6199F863" Ref="R37"  Part="1"
+AR Path="/61996AA1/61A3B341/6199F863" Ref="R42"  Part="1"
+AR Path="/61996AA1/61A3CF51/6199F863" Ref="R47"  Part="1"
+F 0 "R47" H 2892 2104 50  0000 R CNN
 F 1 "30" H 2892 2195 50  0000 R CNN
 F 2 "" H 2950 2150 50  0001 C CNN
@@
 	2500 1950 2950 1950
 $Comp
-L Device:R_Small R?
+L Device:R_Small R23
 U 1 1 619A21A9
 P 3300 1950
-AR Path="/61996AA1/6199D637/619A21A9" Ref="R?"  Part="1"
-AR Path="/61996AA1/61A346F1/619A21A9" Ref="R?"  Part="1"
-AR Path="/61996AA1/61A395F7/619A21A9" Ref="R?"  Part="1"
-AR Path="/61996AA1/61A3A424/619A21A9" Ref="R?"  Part="1"
-AR Path="/61996AA1/61A3B341/619A21A9" Ref="R?"  Part="1"
-AR Path="/61996AA1/61A3CF51/619A21A9" Ref="R?"  Part="1"
-F 0 "R?" V 3104 1950 50  0000 C CNN
+AR Path="/61996AA1/6199D637/619A21A9" Ref="R23"  Part="1"
+AR Path="/61996AA1/61A346F1/619A21A9" Ref="R28"  Part="1"
+AR Path="/61996AA1/61A395F7/619A21A9" Ref="R33"  Part="1"
+AR Path="/61996AA1/61A3A424/619A21A9" Ref="R38"  Part="1"
+AR Path="/61996AA1/61A3B341/619A21A9" Ref="R43"  Part="1"
+AR Path="/61996AA1/61A3CF51/619A21A9" Ref="R48"  Part="1"
+F 0 "R48" V 3104 1950 50  0000 C CNN
 F 1 "330" V 3195 1950 50  0000 C CNN
 F 2 "" H 3300 1950 50  0001 C CNN
@@
 	3550 2400 3400 2400
 $Comp
-L Device:LED_Small D?
+L Device:LED_Small D6
 U 1 1 619A6565
 P 3300 2400
-AR Path="/61996AA1/6199D637/619A6565" Ref="D?"  Part="1"
-AR Path="/61996AA1/61A346F1/619A6565" Ref="D?"  Part="1"
-AR Path="/61996AA1/61A395F7/619A6565" Ref="D?"  Part="1"
-AR Path="/61996AA1/61A3A424/619A6565" Ref="D?"  Part="1"
-AR Path="/61996AA1/61A3B341/619A6565" Ref="D?"  Part="1"
-AR Path="/61996AA1/61A3CF51/619A6565" Ref="D?"  Part="1"
-F 0 "D?" H 3300 2635 50  0000 C CNN
+AR Path="/61996AA1/6199D637/619A6565" Ref="D6"  Part="1"
+AR Path="/61996AA1/61A346F1/619A6565" Ref="D8"  Part="1"
+AR Path="/61996AA1/61A395F7/619A6565" Ref="D10"  Part="1"
+AR Path="/61996AA1/61A3A424/619A6565" Ref="D12"  Part="1"
+AR Path="/61996AA1/61A3B341/619A6565" Ref="D14"  Part="1"
+AR Path="/61996AA1/61A3CF51/619A6565" Ref="D16"  Part="1"
+F 0 "D16" H 3300 2635 50  0000 C CNN
 F 1 "LED_RED" H 3300 2544 50  0000 C CNN
 F 2 "" V 3300 2400 50  0001 C CNN
@@
 Connection ~ 2950 2400
 $Comp
-L Device:Q_NMOS_GSD Q?
+L Device:Q_NMOS_GSD Q2
 U 1 1 619A7C3D
 P 3050 2750
-AR Path="/61996AA1/6199D637/619A7C3D" Ref="Q?"  Part="1"
-AR Path="/61996AA1/61A346F1/619A7C3D" Ref="Q?"  Part="1"
-AR Path="/61996AA1/61A395F7/619A7C3D" Ref="Q?"  Part="1"
-AR Path="/61996AA1/61A3A424/619A7C3D" Ref="Q?"  Part="1"
-AR Path="/61996AA1/61A3B341/619A7C3D" Ref="Q?"  Part="1"
-AR Path="/61996AA1/61A3CF51/619A7C3D" Ref="Q?"  Part="1"
-F 0 "Q?" H 3255 2704 50  0000 L CNN
+AR Path="/61996AA1/6199D637/619A7C3D" Ref="Q2"  Part="1"
+AR Path="/61996AA1/61A346F1/619A7C3D" Ref="Q3"  Part="1"
+AR Path="/61996AA1/61A395F7/619A7C3D" Ref="Q4"  Part="1"
+AR Path="/61996AA1/61A3A424/619A7C3D" Ref="Q5"  Part="1"
+AR Path="/61996AA1/61A3B341/619A7C3D" Ref="Q6"  Part="1"
+AR Path="/61996AA1/61A3CF51/619A7C3D" Ref="Q7"  Part="1"
+F 0 "Q7" H 3255 2704 50  0000 L CNN
 F 1 "Q_NMOS_GSD" H 3255 2795 50  0000 L CNN
 F 2 "" H 3250 2850 50  0001 C CNN
@@
 Connection ~ 2950 3050
 $Comp
-L Device:R_Small R?
+L Device:R_Small R24
 U 1 1 619B0D16
 P 3300 3050
-AR Path="/61996AA1/6199D637/619B0D16" Ref="R?"  Part="1"
-AR Path="/61996AA1/61A346F1/619B0D16" Ref="R?"  Part="1"
-AR Path="/61996AA1/61A395F7/619B0D16" Ref="R?"  Part="1"
-AR Path="/61996AA1/61A3A424/619B0D16" Ref="R?"  Part="1"
-AR Path="/61996AA1/61A3B341/619B0D16" Ref="R?"  Part="1"
-AR Path="/61996AA1/61A3CF51/619B0D16" Ref="R?"  Part="1"
-F 0 "R?" V 3104 3050 50  0000 C CNN
+AR Path="/61996AA1/6199D637/619B0D16" Ref="R24"  Part="1"
+AR Path="/61996AA1/61A346F1/619B0D16" Ref="R29"  Part="1"
+AR Path="/61996AA1/61A395F7/619B0D16" Ref="R34"  Part="1"
+AR Path="/61996AA1/61A3A424/619B0D16" Ref="R39"  Part="1"
+AR Path="/61996AA1/61A3B341/619B0D16" Ref="R44"  Part="1"
+AR Path="/61996AA1/61A3CF51/619B0D16" Ref="R49"  Part="1"
+F 0 "R49" V 3104 3050 50  0000 C CNN
 F 1 "1k" V 3195 3050 50  0000 C CNN
 F 2 "" H 3300 3050 50  0001 C CNN
@@
 Connection ~ 3600 3050
 $Comp
-L Device:D_Zener_Small D?
+L Device:D_Zener_Small D7
 U 1 1 619B293B
 P 3300 3350
-AR Path="/61996AA1/6199D637/619B293B" Ref="D?"  Part="1"
-AR Path="/61996AA1/61A346F1/619B293B" Ref="D?"  Part="1"
-AR Path="/61996AA1/61A395F7/619B293B" Ref="D?"  Part="1"
-AR Path="/61996AA1/61A3A424/619B293B" Ref="D?"  Part="1"
-AR Path="/61996AA1/61A3B341/619B293B" Ref="D?"  Part="1"
-AR Path="/61996AA1/61A3CF51/619B293B" Ref="D?"  Part="1"
-F 0 "D?" H 3300 3143 50  0000 C CNN
+AR Path="/61996AA1/6199D637/619B293B" Ref="D7"  Part="1"
+AR Path="/61996AA1/61A346F1/619B293B" Ref="D9"  Part="1"
+AR Path="/61996AA1/61A395F7/619B293B" Ref="D11"  Part="1"
+AR Path="/61996AA1/61A3A424/619B293B" Ref="D13"  Part="1"
+AR Path="/61996AA1/61A3B341/619B293B" Ref="D15"  Part="1"
+AR Path="/61996AA1/61A3CF51/619B293B" Ref="D17"  Part="1"
+F 0 "D17" H 3300 3143 50  0000 C CNN
 F 1 "D_Zener 9.1V" H 3300 3234 50  0000 C CNN
 F 2 "" V 3300 3350 50  0001 C CNN
@@
 Cell
 $Comp
-L Device:R_Small R?
+L Device:R_Small R25
 U 1 1 619B7EAD
 P 3800 1700
-AR Path="/61996AA1/6199D637/619B7EAD" Ref="R?"  Part="1"
-AR Path="/61996AA1/61A346F1/619B7EAD" Ref="R?"  Part="1"
-AR Path="/61996AA1/61A395F7/619B7EAD" Ref="R?"  Part="1"
-AR Path="/61996AA1/61A3A424/619B7EAD" Ref="R?"  Part="1"
-AR Path="/61996AA1/61A3B341/619B7EAD" Ref="R?"  Part="1"
-AR Path="/61996AA1/61A3CF51/619B7EAD" Ref="R?"  Part="1"
-F 0 "R?" V 3604 1700 50  0000 C CNN
+AR Path="/61996AA1/6199D637/619B7EAD" Ref="R25"  Part="1"
+AR Path="/61996AA1/61A346F1/619B7EAD" Ref="R30"  Part="1"
+AR Path="/61996AA1/61A395F7/619B7EAD" Ref="R35"  Part="1"
+AR Path="/61996AA1/61A3A424/619B7EAD" Ref="R40"  Part="1"
+AR Path="/61996AA1/61A3B341/619B7EAD" Ref="R45"  Part="1"
+AR Path="/61996AA1/61A3CF51/619B7EAD" Ref="R50"  Part="1"
+F 0 "R50" V 3604 1700 50  0000 C CNN
 F 1 "100" V 3695 1700 50  0000 C CNN
 F 2 "" H 3800 1700 50  0001 C CNN
@@
 Cx
 $Comp
-L Device:C_Small C?
+L Device:C_Small C19
 U 1 1 619BEE0A
 P 4000 1900
-AR Path="/61996AA1/6199D637/619BEE0A" Ref="C?"  Part="1"
-AR Path="/61996AA1/61A346F1/619BEE0A" Ref="C?"  Part="1"
-AR Path="/61996AA1/61A395F7/619BEE0A" Ref="C?"  Part="1"
-AR Path="/61996AA1/61A3A424/619BEE0A" Ref="C?"  Part="1"
-AR Path="/61996AA1/61A3B341/619BEE0A" Ref="C?"  Part="1"
-AR Path="/61996AA1/61A3CF51/619BEE0A" Ref="C?"  Part="1"
-F 0 "C?" H 4092 1946 50  0000 L CNN
+AR Path="/61996AA1/6199D637/619BEE0A" Ref="C19"  Part="1"
+AR Path="/61996AA1/61A346F1/619BEE0A" Ref="C20"  Part="1"
+AR Path="/61996AA1/61A395F7/619BEE0A" Ref="C21"  Part="1"
+AR Path="/61996AA1/61A3A424/619BEE0A" Ref="C22"  Part="1"
+AR Path="/61996AA1/61A3B341/619BEE0A" Ref="C23"  Part="1"
+AR Path="/61996AA1/61A3CF51/619BEE0A" Ref="C24"  Part="1"
+F 0 "C24" H 4092 1946 50  0000 L CNN
 F 1 "10nF" H 4092 1855 50  0000 L CNN
 F 2 "" H 4000 1900 50  0001 C CNN
@@
 	4000 2000 4000 2050
 $Comp
-L power:GND #PWR?
+L power:GND #PWR032
 U 1 1 619C00A1
 P 4000 2050
-AR Path="/61996AA1/6199D637/619C00A1" Ref="#PWR?"  Part="1"
-AR Path="/61996AA1/61A346F1/619C00A1" Ref="#PWR?"  Part="1"
-AR Path="/61996AA1/61A395F7/619C00A1" Ref="#PWR?"  Part="1"
-AR Path="/61996AA1/61A3A424/619C00A1" Ref="#PWR?"  Part="1"
-AR Path="/61996AA1/61A3B341/619C00A1" Ref="#PWR?"  Part="1"
-AR Path="/61996AA1/61A3CF51/619C00A1" Ref="#PWR?"  Part="1"
-F 0 "#PWR?" H 4000 1800 50  0001 C CNN
+AR Path="/61996AA1/6199D637/619C00A1" Ref="#PWR032"  Part="1"
+AR Path="/61996AA1/61A346F1/619C00A1" Ref="#PWR033"  Part="1"
+AR Path="/61996AA1/61A395F7/619C00A1" Ref="#PWR034"  Part="1"
+AR Path="/61996AA1/61A3A424/619C00A1" Ref="#PWR035"  Part="1"
+AR Path="/61996AA1/61A3B341/619C00A1" Ref="#PWR036"  Part="1"
+AR Path="/61996AA1/61A3CF51/619C00A1" Ref="#PWR037"  Part="1"
+F 0 "#PWR037" H 4000 1800 50  0001 C CNN
 F 1 "GND" H 4005 1877 50  0000 C CNN
 F 2 "" H 4000 2050 50  0001 C CNN

Commit message: Most of the footprints added
Parts:
- C19: footprint (none) -> Capacitor_SMD:C_0603_1608Metric
- D6: footprint (none) -> LED_SMD:LED_0603_1608Metric
- D7: footprint (none) -> Diode_SMD:D_SMB
- Q2: footprint (none) -> Package_TO_SOT_SMD:SOT-23
- R21, R22: footprint (none) -> Resistor_SMD:R_2512_6332Metric
- R23, R24, R25: footprint (none) -> Resistor_SMD:R_0603_1608Metric
Other:
- moved on the sheet: C24, D16, D17, Q7, R46, R47, R48, R49, R50

Commit message: Thermistors change
Changed lines of the file:
@@
 $Descr A4 11693 8268
 encoding utf-8
-Sheet 8 13
+Sheet 7 13
 Title "Balance part of LTC6810"
 Date ""
@@
 AR Path="/61996AA1/61A3B341/6199E2E8" Ref="R41"  Part="1"
 AR Path="/61996AA1/61A3CF51/6199E2E8" Ref="R46"  Part="1"
-F 0 "R46" H 5592 4004 50  0000 R CNN
+F 0 "R41" H 5592 4004 50  0000 R CNN
 F 1 "30" H 5592 4095 50  0000 R CNN
 F 2 "Resistor_SMD:R_2512_6332Metric" H 5650 4050 50  0001 C CNN
@@
 AR Path="/61996AA1/61A3B341/6199F863" Ref="R42"  Part="1"
 AR Path="/61996AA1/61A3CF51/6199F863" Ref="R47"  Part="1"
-F 0 "R47" H 6042 4004 50  0000 R CNN
+F 0 "R42" H 6042 4004 50  0000 R CNN
 F 1 "30" H 6042 4095 50  0000 R CNN
 F 2 "Resistor_SMD:R_2512_6332Metric" H 6100 4050 50  0001 C CNN
@@
 AR Path="/61996AA1/61A3B341/619A21A9" Ref="R43"  Part="1"
 AR Path="/61996AA1/61A3CF51/619A21A9" Ref="R48"  Part="1"
-F 0 "R48" V 6254 3850 50  0000 C CNN
+F 0 "R43" V 6254 3850 50  0000 C CNN
 F 1 "330" V 6345 3850 50  0000 C CNN
 F 2 "Resistor_SMD:R_0603_1608Metric" H 6450 3850 50  0001 C CNN
@@
 AR Path="/61996AA1/61A3B341/619A6565" Ref="D14"  Part="1"
 AR Path="/61996AA1/61A3CF51/619A6565" Ref="D16"  Part="1"
-F 0 "D16" H 6450 4535 50  0000 C CNN
+F 0 "D14" H 6450 4535 50  0000 C CNN
 F 1 "LED_RED" H 6450 4444 50  0000 C CNN
 F 2 "LED_SMD:LED_0603_1608Metric" V 6450 4300 50  0001 C CNN
@@
 AR Path="/61996AA1/61A3B341/619B0D16" Ref="R44"  Part="1"
 AR Path="/61996AA1/61A3CF51/619B0D16" Ref="R49"  Part="1"
-F 0 "R49" V 6254 4950 50  0000 C CNN
+F 0 "R44" V 6254 4950 50  0000 C CNN
 F 1 "1k" V 6345 4950 50  0000 C CNN
 F 2 "Resistor_SMD:R_0603_1608Metric" H 6450 4950 50  0001 C CNN
@@
 AR Path="/61996AA1/61A3B341/619B293B" Ref="D15"  Part="1"
 AR Path="/61996AA1/61A3CF51/619B293B" Ref="D17"  Part="1"
-F 0 "D17" H 6450 5043 50  0000 C CNN
+F 0 "D15" H 6450 5043 50  0000 C CNN
 F 1 "D_Zener 9.1V" H 6450 5134 50  0000 C CNN
 F 2 "Diode_SMD:D_SMB" V 6450 5250 50  0001 C CNN
@@
 AR Path="/61996AA1/61A3B341/619B7EAD" Ref="R45"  Part="1"
 AR Path="/61996AA1/61A3CF51/619B7EAD" Ref="R50"  Part="1"
-F 0 "R50" V 6754 3600 50  0000 C CNN
+F 0 "R45" V 6754 3600 50  0000 C CNN
 F 1 "100" V 6845 3600 50  0000 C CNN
 F 2 "Resistor_SMD:R_0603_1608Metric" H 6950 3600 50  0001 C CNN
@@
 AR Path="/61996AA1/61A3B341/619BEE0A" Ref="C23"  Part="1"
 AR Path="/61996AA1/61A3CF51/619BEE0A" Ref="C24"  Part="1"
-F 0 "C24" H 7242 3846 50  0000 L CNN
+F 0 "C23" H 7242 3846 50  0000 L CNN
 F 1 "10nF" H 7242 3755 50  0000 L CNN
 F 2 "Capacitor_SMD:C_0603_1608Metric" H 7150 3800 50  0001 C CNN
@@
 AR Path="/61996AA1/61A3B341/619C00A1" Ref="#PWR036"  Part="1"
 AR Path="/61996AA1/61A3CF51/619C00A1" Ref="#PWR037"  Part="1"
-F 0 "#PWR037" H 7150 3700 50  0001 C CNN
+F 0 "#PWR036" H 7150 3700 50  0001 C CNN
 F 1 "GND" H 7155 3777 50  0000 C CNN
 F 2 "" H 7150 3950 50  0001 C CNN
@@
 AR Path="/61996AA1/61A3B341/619A7C3D" Ref="Q6"  Part="1"
 AR Path="/61996AA1/61A3CF51/619A7C3D" Ref="Q7"  Part="1"
-F 0 "Q7" H 6405 4604 50  0000 L CNN
+F 0 "Q6" H 6405 4604 50  0000 L CNN
 F 1 "Q_NMOS_GSD" H 6405 4695 50  0000 L CNN
 F 2 "Package_TO_SOT_SMD:SOT-23" H 6400 4750 50  0001 C CNN

Commit message: PCB update
Parts changed due to smaller footprints
Parts:
- D7: footprint Diode_SMD:D_SMB -> Diode_SMD:D_SOD-323; Part Number (none) -> BZX384-C9V1.115
Changed lines of the file:
@@
 $Descr A4 11693 8268
 encoding utf-8
-Sheet 7 13
+Sheet 4 13
 Title "Balance part of LTC6810"
 Date ""
@@
 AR Path="/61996AA1/61A3B341/6199E2E8" Ref="R41"  Part="1"
 AR Path="/61996AA1/61A3CF51/6199E2E8" Ref="R46"  Part="1"
-F 0 "R41" H 5592 4004 50  0000 R CNN
+F 0 "R46" H 5592 4004 50  0000 R CNN
 F 1 "30" H 5592 4095 50  0000 R CNN
 F 2 "Resistor_SMD:R_2512_6332Metric" H 5650 4050 50  0001 C CNN
@@
 AR Path="/61996AA1/61A3B341/6199F863" Ref="R42"  Part="1"
 AR Path="/61996AA1/61A3CF51/6199F863" Ref="R47"  Part="1"
-F 0 "R42" H 6042 4004 50  0000 R CNN
+F 0 "R47" H 6042 4004 50  0000 R CNN
 F 1 "30" H 6042 4095 50  0000 R CNN
 F 2 "Resistor_SMD:R_2512_6332Metric" H 6100 4050 50  0001 C CNN
@@
 AR Path="/61996AA1/61A3B341/619A21A9" Ref="R43"  Part="1"
 AR Path="/61996AA1/61A3CF51/619A21A9" Ref="R48"  Part="1"
-F 0 "R43" V 6254 3850 50  0000 C CNN
+F 0 "R48" V 6254 3850 50  0000 C CNN
 F 1 "330" V 6345 3850 50  0000 C CNN
 F 2 "Resistor_SMD:R_0603_1608Metric" H 6450 3850 50  0001 C CNN
@@
 AR Path="/61996AA1/61A3B341/619A6565" Ref="D14"  Part="1"
 AR Path="/61996AA1/61A3CF51/619A6565" Ref="D16"  Part="1"
-F 0 "D14" H 6450 4535 50  0000 C CNN
+F 0 "D16" H 6450 4535 50  0000 C CNN
 F 1 "LED_RED" H 6450 4444 50  0000 C CNN
 F 2 "LED_SMD:LED_0603_1608Metric" V 6450 4300 50  0001 C CNN
@@
 AR Path="/61996AA1/61A3B341/619B0D16" Ref="R44"  Part="1"
 AR Path="/61996AA1/61A3CF51/619B0D16" Ref="R49"  Part="1"
-F 0 "R44" V 6254 4950 50  0000 C CNN
+F 0 "R49" V 6254 4950 50  0000 C CNN
 F 1 "1k" V 6345 4950 50  0000 C CNN
 F 2 "Resistor_SMD:R_0603_1608Metric" H 6450 4950 50  0001 C CNN
@@
 AR Path="/61996AA1/61A3B341/619B293B" Ref="D15"  Part="1"
 AR Path="/61996AA1/61A3CF51/619B293B" Ref="D17"  Part="1"
-F 0 "D15" H 6450 5043 50  0000 C CNN
+F 0 "D17" H 6450 5043 50  0000 C CNN
 F 1 "D_Zener 9.1V" H 6450 5134 50  0000 C CNN
-F 2 "Diode_SMD:D_SMB" V 6450 5250 50  0001 C CNN
+F 2 "Diode_SMD:D_SOD-323" V 6450 5250 50  0001 C CNN
 F 3 "~" V 6450 5250 50  0001 C CNN
+F 4 "BZX384-C9V1.115" H 6450 5250 50  0001 C CNN "Part Number"
 	1    6450 5250
 	-1   0    0    1
@@
 AR Path="/61996AA1/61A3B341/619B7EAD" Ref="R45"  Part="1"
 AR Path="/61996AA1/61A3CF51/619B7EAD" Ref="R50"  Part="1"
-F 0 "R45" V 6754 3600 50  0000 C CNN
+F 0 "R50" V 6754 3600 50  0000 C CNN
 F 1 "100" V 6845 3600 50  0000 C CNN
 F 2 "Resistor_SMD:R_0603_1608Metric" H 6950 3600 50  0001 C CNN
@@
 AR Path="/61996AA1/61A3B341/619BEE0A" Ref="C23"  Part="1"
 AR Path="/61996AA1/61A3CF51/619BEE0A" Ref="C24"  Part="1"
-F 0 "C23" H 7242 3846 50  0000 L CNN
+F 0 "C24" H 7242 3846 50  0000 L CNN
 F 1 "10nF" H 7242 3755 50  0000 L CNN
 F 2 "Capacitor_SMD:C_0603_1608Metric" H 7150 3800 50  0001 C CNN
@@
 AR Path="/61996AA1/61A3B341/619C00A1" Ref="#PWR036"  Part="1"
 AR Path="/61996AA1/61A3CF51/619C00A1" Ref="#PWR037"  Part="1"
-F 0 "#PWR036" H 7150 3700 50  0001 C CNN
+F 0 "#PWR037" H 7150 3700 50  0001 C CNN
 F 1 "GND" H 7155 3777 50  0000 C CNN
 F 2 "" H 7150 3950 50  0001 C CNN
@@
 AR Path="/61996AA1/61A3B341/619A7C3D" Ref="Q6"  Part="1"
 AR Path="/61996AA1/61A3CF51/619A7C3D" Ref="Q7"  Part="1"
-F 0 "Q6" H 6405 4604 50  0000 L CNN
+F 0 "Q7" H 6405 4604 50  0000 L CNN
 F 1 "Q_NMOS_GSD" H 6405 4695 50  0000 L CNN
 F 2 "Package_TO_SOT_SMD:SOT-23" H 6400 4750 50  0001 C CNN

Commit message: PCB Layout Update
Some work on PCB Layout
+ AS214-97PN (connector) 3D model added
Changed lines of the file:
@@
 $Descr A4 11693 8268
 encoding utf-8
-Sheet 4 13
+Sheet 3 13
 Title "Balance part of LTC6810"
 Date ""
@@
 AR Path="/61996AA1/61A3B341/6199E2E8" Ref="R41"  Part="1"
 AR Path="/61996AA1/61A3CF51/6199E2E8" Ref="R46"  Part="1"
-F 0 "R46" H 5592 4004 50  0000 R CNN
+F 0 "R21" H 5592 4004 50  0000 R CNN
 F 1 "30" H 5592 4095 50  0000 R CNN
 F 2 "Resistor_SMD:R_2512_6332Metric" H 5650 4050 50  0001 C CNN
@@
 AR Path="/61996AA1/61A3B341/6199F863" Ref="R42"  Part="1"
 AR Path="/61996AA1/61A3CF51/6199F863" Ref="R47"  Part="1"
-F 0 "R47" H 6042 4004 50  0000 R CNN
+F 0 "R22" H 6042 4004 50  0000 R CNN
 F 1 "30" H 6042 4095 50  0000 R CNN
 F 2 "Resistor_SMD:R_2512_6332Metric" H 6100 4050 50  0001 C CNN
@@
 AR Path="/61996AA1/61A3B341/619A21A9" Ref="R43"  Part="1"
 AR Path="/61996AA1/61A3CF51/619A21A9" Ref="R48"  Part="1"
-F 0 "R48" V 6254 3850 50  0000 C CNN
+F 0 "R23" V 6254 3850 50  0000 C CNN
 F 1 "330" V 6345 3850 50  0000 C CNN
 F 2 "Resistor_SMD:R_0603_1608Metric" H 6450 3850 50  0001 C CNN
@@
 AR Path="/61996AA1/61A3B341/619A6565" Ref="D14"  Part="1"
 AR Path="/61996AA1/61A3CF51/619A6565" Ref="D16"  Part="1"
-F 0 "D16" H 6450 4535 50  0000 C CNN
+F 0 "D6" H 6450 4535 50  0000 C CNN
 F 1 "LED_RED" H 6450 4444 50  0000 C CNN
 F 2 "LED_SMD:LED_0603_1608Metric" V 6450 4300 50  0001 C CNN
@@
 AR Path="/61996AA1/61A3B341/619B0D16" Ref="R44"  Part="1"
 AR Path="/61996AA1/61A3CF51/619B0D16" Ref="R49"  Part="1"
-F 0 "R49" V 6254 4950 50  0000 C CNN
+F 0 "R24" V 6254 4950 50  0000 C CNN
 F 1 "1k" V 6345 4950 50  0000 C CNN
 F 2 "Resistor_SMD:R_0603_1608Metric" H 6450 4950 50  0001 C CNN
@@
 AR Path="/61996AA1/61A3B341/619B293B" Ref="D15"  Part="1"
 AR Path="/61996AA1/61A3CF51/619B293B" Ref="D17"  Part="1"
-F 0 "D17" H 6450 5043 50  0000 C CNN
+F 0 "D7" H 6450 5043 50  0000 C CNN
 F 1 "D_Zener 9.1V" H 6450 5134 50  0000 C CNN
 F 2 "Diode_SMD:D_SOD-323" V 6450 5250 50  0001 C CNN
@@
 AR Path="/61996AA1/61A3B341/619B7EAD" Ref="R45"  Part="1"
 AR Path="/61996AA1/61A3CF51/619B7EAD" Ref="R50"  Part="1"
-F 0 "R50" V 6754 3600 50  0000 C CNN
+F 0 "R25" V 6754 3600 50  0000 C CNN
 F 1 "100" V 6845 3600 50  0000 C CNN
 F 2 "Resistor_SMD:R_0603_1608Metric" H 6950 3600 50  0001 C CNN
@@
 AR Path="/61996AA1/61A3B341/619BEE0A" Ref="C23"  Part="1"
 AR Path="/61996AA1/61A3CF51/619BEE0A" Ref="C24"  Part="1"
-F 0 "C24" H 7242 3846 50  0000 L CNN
+F 0 "C19" H 7242 3846 50  0000 L CNN
 F 1 "10nF" H 7242 3755 50  0000 L CNN
 F 2 "Capacitor_SMD:C_0603_1608Metric" H 7150 3800 50  0001 C CNN
@@
 AR Path="/61996AA1/61A3B341/619C00A1" Ref="#PWR036"  Part="1"
 AR Path="/61996AA1/61A3CF51/619C00A1" Ref="#PWR037"  Part="1"
-F 0 "#PWR037" H 7150 3700 50  0001 C CNN
+F 0 "#PWR032" H 7150 3700 50  0001 C CNN
 F 1 "GND" H 7155 3777 50  0000 C CNN
 F 2 "" H 7150 3950 50  0001 C CNN
@@
 AR Path="/61996AA1/61A3B341/619A7C3D" Ref="Q6"  Part="1"
 AR Path="/61996AA1/61A3CF51/619A7C3D" Ref="Q7"  Part="1"
-F 0 "Q7" H 6405 4604 50  0000 L CNN
+F 0 "Q2" H 6405 4604 50  0000 L CNN
 F 1 "Q_NMOS_GSD" H 6405 4695 50  0000 L CNN
 F 2 "Package_TO_SOT_SMD:SOT-23" H 6400 4750 50  0001 C CNN

Commit message: PCB Layout Update 3
Parts:
- R21, R22: Part Number (none) -> CHP2512AFX-10R0ELF
Connections:
- net GND renamed GNDPWR
Changed lines of the file:
@@
 $Descr A4 11693 8268
 encoding utf-8
-Sheet 3 13
+Sheet 5 13
 Title "Balance part of LTC6810"
 Date ""
@@
 F 2 "Resistor_SMD:R_2512_6332Metric" H 5650 4050 50  0001 C CNN
 F 3 "~" H 5650 4050 50  0001 C CNN
+F 4 "CHP2512AFX-10R0ELF" H 5650 4050 50  0001 C CNN "Part Number"
 	1    5650 4050
 	1    0    0    1
@@
 F 2 "Resistor_SMD:R_2512_6332Metric" H 6100 4050 50  0001 C CNN
 F 3 "~" H 6100 4050 50  0001 C CNN
+F 4 "CHP2512AFX-10R0ELF" H 6100 4050 50  0001 C CNN "Part Number"
 	1    6100 4050
 	1    0    0    1
@@
 Wire Wire Line
 	5150 4950 5150 3600
-Text HLabel 6100 3500 0    50   Input ~ 0
+Text HLabel 6100 3700 0    50   Input ~ 0
 PreviousBalance
-Wire Wire Line
-	6100 3500 6100 3850
 Wire Wire Line
 	7050 3600 7150 3600
@@
 Wire Wire Line
 	7150 3900 7150 3950
-$Comp
-L power:GND #PWR032
-U 1 1 619C00A1
-P 7150 3950
-AR Path="/61996AA1/6199D637/619C00A1" Ref="#PWR032"  Part="1"
-AR Path="/61996AA1/61A346F1/619C00A1" Ref="#PWR033"  Part="1"
-AR Path="/61996AA1/61A395F7/619C00A1" Ref="#PWR034"  Part="1"
-AR Path="/61996AA1/61A3A424/619C00A1" Ref="#PWR035"  Part="1"
-AR Path="/61996AA1/61A3B341/619C00A1" Ref="#PWR036"  Part="1"
-AR Path="/61996AA1/61A3CF51/619C00A1" Ref="#PWR037"  Part="1"
-F 0 "#PWR032" H 7150 3700 50  0001 C CNN
-F 1 "GND" H 7155 3777 50  0000 C CNN
-F 2 "" H 7150 3950 50  0001 C CNN
-F 3 "" H 7150 3950 50  0001 C CNN
-	1    7150 3950
-	1    0    0    -1
-$EndComp
 Text HLabel 6100 5450 2    50   Input ~ 0
 NextBalance
@@
 	-1   0    0    -1
 $EndComp
+$Comp
+L power:GNDPWR #PWR?
+U 1 1 61F1BB4A
+P 7150 3950
+AR Path="/61996AA1/61F1BB4A" Ref="#PWR?"  Part="1"
+AR Path="/61996AA1/61A346F1/61F1BB4A" Ref="#PWR0113"  Part="1"
+AR Path="/61996AA1/6199D637/61F1BB4A" Ref="#PWR0112"  Part="1"
+AR Path="/61996AA1/61A395F7/61F1BB4A" Ref="#PWR0114"  Part="1"
+AR Path="/61996AA1/61A3A424/61F1BB4A" Ref="#PWR0115"  Part="1"
+AR Path="/61996AA1/61A3B341/61F1BB4A" Ref="#PWR0116"  Part="1"
+AR Path="/61996AA1/61A3CF51/61F1BB4A" Ref="#PWR0117"  Part="1"
+F 0 "#PWR0112" H 7150 3750 50  0001 C CNN
+F 1 "GNDPWR" H 7154 3796 50  0000 C CNN
+F 2 "" H 7150 3900 50  0001 C CNN
+F 3 "" H 7150 3900 50  0001 C CNN
+	1    7150 3950
+	1    0    0    -1
+$EndComp
+Wire Wire Line
+	6100 3850 6100 3700
 $EndSCHEMATC
