File: HARDWARE/BMS_LV_2022/CAN.sch (KiCad schematic (older format))
At the start: 9 parts, among them U3 ATA6561-GAQW-N

Commit message: Thermistors change
Parts:
- R3: value 120R -> 120
Changed lines of the file:
@@
 AR Path="/61F4D531/61A896F4" Ref="R4"  Part="1"
 F 0 "R4" H 8970 4146 50  0000 L CNN
-F 1 "120R" H 8970 4055 50  0000 L CNN
+F 1 "120" H 8970 4055 50  0000 L CNN
 F 2 "Resistor_SMD:R_0603_1608Metric" V 8830 4100 50  0001 C CNN
 F 3 "~" H 8900 4100 50  0001 C CNN

Commit message: PCB Routing Update
Parts:
- U3: footprint Package_DFN_QFN:DFN-8-1EP_3x3mm_P0.65mm_EP1.55x2.4mm -> Package_SO:SOIC-8_3.9x4.9mm_P1.27mm
Changed lines of the file:
@@
 EESchema Schematic File Version 4
-LIBS:BMS_LV_2022-cache
-EELAYER 29 0
+EELAYER 30 0
 EELAYER END
 $Descr A4 11693 8268
@@
 F 0 "U4" H 6100 4450 50  0000 C CNN
 F 1 "ATA6561-GAQW-N" H 6200 4350 50  0000 C CNN
-F 2 "Package_DFN_QFN:DFN-8-1EP_3x3mm_P0.65mm_EP1.55x2.4mm" H 5700 3450 50  0001 C CIN
+F 2 "Package_SO:SOIC-8_3.9x4.9mm_P1.27mm" H 5700 3450 50  0001 C CIN
 F 3 "https://pl.mouser.com/datasheet/2/268/ATA6560_ATA6561_High_Speed_CAN_Transceiver_DS20005-1384933.pdf" H 5700 3950 50  0001 C CNN
 	1    5700 3950
