File: HARDWARE/BMS_LV_2022/LTC6810.sch (KiCad schematic (older format))
At the start: 28 parts

Commit message: Hardware Update 2
First verison of the scheme finished
+Power section
+eFuse section
+Current Sensor section
+Connectors section
+Debug LEDs
+STM32L4P5RET6 all signals configuration
Parts:
- added R? (x4): 2.2k, symbol Device:R_Small
Connections:
- net labels added: +3.3V
- wire segments 138 -> 159
Other:
- moved on the sheet: J?
Changed lines of the file:
@@
 $Descr A4 11693 8268
 encoding utf-8
-Sheet 2 10
-Title ""
+Sheet 2 13
+Title "LTC6810 Application"
 Date ""
 Rev ""
@@
 Wire Wire Line
 	3750 5950 3850 5950
-Text HLabel 6650 2600 2    50   Input ~ 0
+Text HLabel 6900 2600 2    50   Input ~ 0
 MOSI
-Text HLabel 6650 2700 2    50   Input ~ 0
+Text HLabel 6900 2700 2    50   Input ~ 0
 MISO
 $Comp
@@
 U 1 1 61AF3C75
 P 7000 3000
-F 0 "R?" V 6804 3000 50  0000 C CNN
-F 1 "10k" V 6895 3000 50  0000 C CNN
+F 0 "R?" V 6950 2850 50  0000 C CNN
+F 1 "10k" V 7050 2850 50  0000 C CNN
 F 2 "" H 7000 3000 50  0001 C CNN
 F 3 "~" H 7000 3000 50  0001 C CNN
@@
 	0    1    1    0
 $EndComp
-Text HLabel 6650 2800 2    50   Input ~ 0
+Text HLabel 6900 2800 2    50   Input ~ 0
 SCK
-Text HLabel 6650 2900 2    50   Input ~ 0
+Text HLabel 6900 2900 2    50   Input ~ 0
 CS
 $Comp
@@
 L Connector:Conn_01x01_Female J?
 U 1 1 61AB3B1A
-P 3300 5950
-F 0 "J?" H 3700 6050 50  0000 C CNN
-F 1 "Conn_01x01_Female" H 3700 5950 50  0000 C CNN
-F 2 "" H 3300 5950 50  0001 C CNN
-F 3 "~" H 3300 5950 50  0001 C CNN
-	1    3300 5950
+P 3250 5950
+F 0 "J?" H 3650 6050 50  0000 C CNN
+F 1 "Conn_01x01_Female" H 3650 5950 50  0000 C CNN
+F 2 "" H 3250 5950 50  0001 C CNN
+F 3 "~" H 3250 5950 50  0001 C CNN
+	1    3250 5950
 	-1   0    0    -1
 $EndComp
@@
 L Connector:Conn_01x01_Female J?
 U 1 1 61AAFFF2
-P 3300 5350
-F 0 "J?" H 3700 5450 50  0000 C CNN
-F 1 "Conn_01x01_Female" H 3700 5350 50  0000 C CNN
-F 2 "" H 3300 5350 50  0001 C CNN
-F 3 "~" H 3300 5350 50  0001 C CNN
-	1    3300 5350
+P 3250 5350
+F 0 "J?" H 3650 5450 50  0000 C CNN
+F 1 "Conn_01x01_Female" H 3650 5350 50  0000 C CNN
+F 2 "" H 3250 5350 50  0001 C CNN
+F 3 "~" H 3250 5350 50  0001 C CNN
+	1    3250 5350
 	-1   0    0    -1
 $EndComp
@@
 L Connector:Conn_01x01_Female J?
 U 1 1 61AAC32A
-P 3300 4750
-F 0 "J?" H 3700 4850 50  0000 C CNN
-F 1 "Conn_01x01_Female" H 3700 4750 50  0000 C CNN
-F 2 "" H 3300 4750 50  0001 C CNN
-F 3 "~" H 3300 4750 50  0001 C CNN
-	1    3300 4750
+P 3250 4750
+F 0 "J?" H 3650 4850 50  0000 C CNN
+F 1 "Conn_01x01_Female" H 3650 4750 50  0000 C CNN
+F 2 "" H 3250 4750 50  0001 C CNN
+F 3 "~" H 3250 4750 50  0001 C CNN
+	1    3250 4750
 	-1   0    0    -1
 $EndComp
@@
 L Connector:Conn_01x01_Female J?
 U 1 1 61AA88B9
-P 3300 4150
-F 0 "J?" H 3700 4250 50  0000 C CNN
-F 1 "Conn_01x01_Female" H 3700 4150 50  0000 C CNN
-F 2 "" H 3300 4150 50  0001 C CNN
-F 3 "~" H 3300 4150 50  0001 C CNN
-	1    3300 4150
+P 3250 4150
+F 0 "J?" H 3650 4250 50  0000 C CNN
+F 1 "Conn_01x01_Female" H 3650 4150 50  0000 C CNN
+F 2 "" H 3250 4150 50  0001 C CNN
+F 3 "~" H 3250 4150 50  0001 C CNN
+	1    3250 4150
 	-1   0    0    -1
 $EndComp
@@
 L Connector:Conn_01x01_Female J?
 U 1 1 61A9D24A
-P 3300 3550
-F 0 "J?" H 3700 3650 50  0000 C CNN
-F 1 "Conn_01x01_Female" H 3700 3550 50  0000 C CNN
-F 2 "" H 3300 3550 50  0001 C CNN
-F 3 "~" H 3300 3550 50  0001 C CNN
-	1    3300 3550
+P 3250 3550
+F 0 "J?" H 3650 3650 50  0000 C CNN
+F 1 "Conn_01x01_Female" H 3650 3550 50  0000 C CNN
+F 2 "" H 3250 3550 50  0001 C CNN
+F 3 "~" H 3250 3550 50  0001 C CNN
+	1    3250 3550
 	-1   0    0    -1
 $EndComp
@@
 L Connector:Conn_01x01_Female J?
 U 1 1 61A336C9
-P 3300 2950
-F 0 "J?" H 3700 3050 50  0000 C CNN
-F 1 "Conn_01x01_Female" H 3700 2950 50  0000 C CNN
-F 2 "" H 3300 2950 50  0001 C CNN
-F 3 "~" H 3300 2950 50  0001 C CNN
-	1    3300 2950
+P 3250 2950
+F 0 "J?" H 3650 3050 50  0000 C CNN
+F 1 "Conn_01x01_Female" H 3650 2950 50  0000 C CNN
+F 2 "" H 3250 2950 50  0001 C CNN
+F 3 "~" H 3250 2950 50  0001 C CNN
+	1    3250 2950
 	-1   0    0    -1
 $EndComp
@@
 L Connector:Conn_01x01_Female J?
 U 1 1 61A1B6B1
-P 3300 2300
-F 0 "J?" H 3700 2400 50  0000 C CNN
-F 1 "Conn_01x01_Female" H 3700 2300 50  0000 C CNN
-F 2 "" H 3300 2300 50  0001 C CNN
-F 3 "~" H 3300 2300 50  0001 C CNN
-	1    3300 2300
-	-1   0    0    -1
-$EndComp
+P 3250 2300
+F 0 "J?" H 3650 2400 50  0000 C CNN
+F 1 "Conn_01x01_Female" H 3650 2300 50  0000 C CNN
+F 2 "" H 3250 2300 50  0001 C CNN
+F 3 "~" H 3250 2300 50  0001 C CNN
+	1    3250 2300
+	-1   0    0    -1
+$EndComp
+Text Label 6700 2900 0    50   ~ 0
+CS
+Text Label 6700 2800 0    50   ~ 0
+SCK
+Text Label 6700 2700 0    50   ~ 0
+MISO
+Text Label 6700 2600 0    50   ~ 0
+MOSI
+Wire Wire Line
+	6900 2600 6650 2600
+Wire Wire Line
+	6650 2700 6900 2700
+Wire Wire Line
+	6650 2800 6900 2800
+Wire Wire Line
+	6650 2900 6900 2900
+Wire Wire Line
+	7550 4850 7700 4850
+Connection ~ 7550 4850
+Wire Wire Line
+	7550 4800 7550 4850
+Wire Wire Line
+	7700 4850 8000 4850
+Connection ~ 7700 4850
+Wire Wire Line
+	7400 4850 7550 4850
+Connection ~ 7400 4850
+Wire Wire Line
+	7100 4850 7400 4850
+$Comp
+L Device:R_Small R?
+U 1 1 61D19CAB
+P 8000 4950
+F 0 "R?" H 8059 4996 50  0000 L CNN
+F 1 "2.2k" H 8059 4905 50  0000 L CNN
+F 2 "" H 8000 4950 50  0001 C CNN
+F 3 "~" H 8000 4950 50  0001 C CNN
+	1    8000 4950
+	-1   0    0    1
+$EndComp
+$Comp
+L Device:R_Small R?
+U 1 1 61D14087
+P 7700 4950
+F 0 "R?" H 7759 4996 50  0000 L CNN
+F 1 "2.2k" H 7759 4905 50  0000 L CNN
+F 2 "" H 7700 4950 50  0001 C CNN
+F 3 "~" H 7700 4950 50  0001 C CNN
+	1    7700 4950
+	-1   0    0    1
+$EndComp
+$Comp
+L Device:R_Small R?
+U 1 1 61D0E598
+P 7400 4950
+F 0 "R?" H 7459 4996 50  0000 L CNN
+F 1 "2.2k" H 7459 4905 50  0000 L CNN
+F 2 "" H 7400 4950 50  0001 C CNN
+F 3 "~" H 7400 4950 50  0001 C CNN
+	1    7400 4950
+	-1   0    0    1
+$EndComp
+$Comp
+L Device:R_Small R?
+U 1 1 61D0640A
+P 7100 4950
+F 0 "R?" H 7159 4996 50  0000 L CNN
+F 1 "2.2k" H 7159 4905 50  0000 L CNN
+F 2 "" H 7100 4950 50  0001 C CNN
+F 3 "~" H 7100 4950 50  0001 C CNN
+	1    7100 4950
+	-1   0    0    1
+$EndComp
+$Comp
+L power:+3.3V #PWR?
+U 1 1 61CFD8CD
+P 7550 4800
+F 0 "#PWR?" H 7550 4650 50  0001 C CNN
+F 1 "+3.3V" H 7565 4973 50  0000 C CNN
+F 2 "" H 7550 4800 50  0001 C CNN
+F 3 "" H 7550 4800 50  0001 C CNN
+	1    7550 4800
+	1    0    0    -1
+$EndComp
+Text Label 7100 5100 3    50   ~ 0
+MOSI
+Wire Wire Line
+	7100 5050 7100 5100
+Text Label 7400 5100 3    50   ~ 0
+MISO
+Wire Wire Line
+	7400 5050 7400 5100
+Text Label 7700 5100 3    50   ~ 0
+SCK
+Wire Wire Line
+	7700 5050 7700 5100
+Text Label 8000 5100 3    50   ~ 0
+CS
+Wire Wire Line
+	8000 5100 8000 5050
+Wire Wire Line
+	3500 2300 3500 2250
+Wire Wire Line
+	3500 2300 3450 2300
+Wire Wire Line
+	3450 5950 3500 5950
+Wire Wire Line
+	3450 5350 3500 5350
+Connection ~ 3500 5350
+Wire Wire Line
+	3450 4750 3500 4750
+Connection ~ 3500 4750
+Wire Wire Line
+	3450 4150 3500 4150
+Connection ~ 3500 4150
+Wire Wire Line
+	3450 3550 3500 3550
+Wire Wire Line
+	3450 2950 3500 2950
 $Comp
 L power:+24V #PWR?
-U 1 1 61A1A4FA
-P 3500 2300
-F 0 "#PWR?" H 3500 2150 50  0001 C CNN
-F 1 "+24V" H 3515 2473 50  0000 C CNN
-F 2 "" H 3500 2300 50  0001 C CNN
-F 3 "" H 3500 2300 50  0001 C CNN
-	1    3500 2300
-	1    0    0    -1
-$EndComp
+U 1 1 622C9690
+P 3500 2250
+F 0 "#PWR?" H 3500 2100 50  0001 C CNN
+F 1 "+24V" H 3515 2423 50  0000 C CNN
+F 2 "" H 3500 2250 50  0001 C CNN
+F 3 "" H 3500 2250 50  0001 C CNN
+	1    3500 2250
+	1    0    0    -1
+$EndComp

Commit message: Hardware update; -changes after team review;
Parts:
- C?: value C_Small -> 1uF
- C?: value C_Small -> 10nF
- C? (x3): value 1u -> 1uF
- C?: value 0.1u -> 0.1uF
- LTC6810?: symbol LTC6810-1:LTC6810-1 -> BMS_LV_2022-rescue:LTC6810-1-LTC6810-1
- R? (x2): value R_Small -> 100
Changed lines of the file:
@@
 P 4650 1900
 F 0 "C?" H 4742 1946 50  0000 L CNN
-F 1 "C_Small" H 4742 1855 50  0000 L CNN
+F 1 "1uF" H 4742 1855 50  0000 L CNN
 F 2 "" H 4650 1900 50  0001 C CNN
 F 3 "~" H 4650 1900 50  0001 C CNN
@@
 P 4350 1800
 F 0 "R?" V 4154 1800 50  0000 C CNN
-F 1 "R_Small" V 4245 1800 50  0000 C CNN
+F 1 "100" V 4245 1800 50  0000 C CNN
 F 2 "" H 4350 1800 50  0001 C CNN
 F 3 "~" H 4350 1800 50  0001 C CNN
@@
 P 4350 2300
 F 0 "R?" V 4154 2300 50  0000 C CNN
-F 1 "R_Small" V 4245 2300 50  0000 C CNN
+F 1 "100" V 4245 2300 50  0000 C CNN
 F 2 "" H 4350 2300 50  0001 C CNN
 F 3 "~" H 4350 2300 50  0001 C CNN
@@
 P 4650 2400
 F 0 "C?" H 4742 2446 50  0000 L CNN
-F 1 "C_Small" H 4742 2355 50  0000 L CNN
+F 1 "10nF" H 4742 2355 50  0000 L CNN
 F 2 "" H 4650 2400 50  0001 C CNN
 F 3 "~" H 4650 2400 50  0001 C CNN
@@
 P 6900 3800
 F 0 "C?" H 6992 3846 50  0000 L CNN
-F 1 "1u" H 6992 3755 50  0000 L CNN
+F 1 "1uF" H 6992 3755 50  0000 L CNN
 F 2 "" H 6900 3800 50  0001 C CNN
 F 3 "~" H 6900 3800 50  0001 C CNN
@@
 P 7200 3800
 F 0 "C?" H 7292 3846 50  0000 L CNN
-F 1 "1u" H 7292 3755 50  0000 L CNN
+F 1 "1uF" H 7292 3755 50  0000 L CNN
 F 2 "" H 7200 3800 50  0001 C CNN
 F 3 "~" H 7200 3800 50  0001 C CNN
@@
 P 7500 3800
 F 0 "C?" H 7592 3846 50  0000 L CNN
-F 1 "1u" H 7592 3755 50  0000 L CNN
+F 1 "1uF" H 7592 3755 50  0000 L CNN
 F 2 "" H 7500 3800 50  0001 C CNN
 F 3 "~" H 7500 3800 50  0001 C CNN
@@
 P 8100 3150
 F 0 "C?" V 7871 3150 50  0000 C CNN
-F 1 "0.1u" V 7962 3150 50  0000 C CNN
+F 1 "0.1uF" V 7962 3150 50  0000 C CNN
 F 2 "" H 8100 3150 50  0001 C CNN
 F 3 "~" H 8100 3150 50  0001 C CNN
@@
 $EndComp
 $Comp
-L LTC6810-1:LTC6810-1 LTC6810?
+L BMS_LV_2022-rescue:LTC6810-1-LTC6810-1 LTC6810?
 U 1 1 61D92574
 P 6950 4600
@@
 $EndComp
 Connection ~ 3500 2300
+Text Label 6700 2900 0    50   ~ 0
+CS
+Text Label 6700 2800 0    50   ~ 0
+SCK
+Text Label 6700 2700 0    50   ~ 0
+MISO
+Text Label 6700 2600 0    50   ~ 0
+MOSI
+Wire Wire Line
+	6900 2600 6650 2600
+Wire Wire Line
+	6650 2700 6900 2700
+Wire Wire Line
+	6650 2800 6900 2800
+Wire Wire Line
+	6650 2900 6900 2900
+Wire Wire Line
+	7550 4850 7700 4850
+Connection ~ 7550 4850
+Wire Wire Line
+	7550 4800 7550 4850
+Wire Wire Line
+	7700 4850 8000 4850
+Connection ~ 7700 4850
+Wire Wire Line
+	7400 4850 7550 4850
+Connection ~ 7400 4850
+Wire Wire Line
+	7100 4850 7400 4850
+$Comp
+L Device:R_Small R?
+U 1 1 61D19CAB
+P 8000 4950
+F 0 "R?" H 8059 4996 50  0000 L CNN
+F 1 "2.2k" H 8059 4905 50  0000 L CNN
+F 2 "" H 8000 4950 50  0001 C CNN
+F 3 "~" H 8000 4950 50  0001 C CNN
+	1    8000 4950
+	-1   0    0    1
+$EndComp
+$Comp
+L Device:R_Small R?
+U 1 1 61D14087
+P 7700 4950
+F 0 "R?" H 7759 4996 50  0000 L CNN
+F 1 "2.2k" H 7759 4905 50  0000 L CNN
+F 2 "" H 7700 4950 50  0001 C CNN
+F 3 "~" H 7700 4950 50  0001 C CNN
+	1    7700 4950
+	-1   0    0    1
+$EndComp
+$Comp
+L Device:R_Small R?
+U 1 1 61D0E598
+P 7400 4950
+F 0 "R?" H 7459 4996 50  0000 L CNN
+F 1 "2.2k" H 7459 4905 50  0000 L CNN
+F 2 "" H 7400 4950 50  0001 C CNN
+F 3 "~" H 7400 4950 50  0001 C CNN
+	1    7400 4950
+	-1   0    0    1
+$EndComp
+$Comp
+L Device:R_Small R?
+U 1 1 61D0640A
+P 7100 4950
+F 0 "R?" H 7159 4996 50  0000 L CNN
+F 1 "2.2k" H 7159 4905 50  0000 L CNN
+F 2 "" H 7100 4950 50  0001 C CNN
+F 3 "~" H 7100 4950 50  0001 C CNN
+	1    7100 4950
+	-1   0    0    1
+$EndComp
+$Comp
+L power:+3.3V #PWR?
+U 1 1 61CFD8CD
+P 7550 4800
+F 0 "#PWR?" H 7550 4650 50  0001 C CNN
+F 1 "+3.3V" H 7565 4973 50  0000 C CNN
+F 2 "" H 7550 4800 50  0001 C CNN
+F 3 "" H 7550 4800 50  0001 C CNN
+	1    7550 4800
+	1    0    0    -1
+$EndComp
+Text Label 7100 5100 3    50   ~ 0
+MOSI
+Wire Wire Line
+	7100 5050 7100 5100
+Text Label 7400 5100 3    50   ~ 0
+MISO
+Wire Wire Line
+	7400 5050 7400 5100
+Text Label 7700 5100 3    50   ~ 0
+SCK
+Wire Wire Line
+	7700 5050 7700 5100
+Text Label 8000 5100 3    50   ~ 0
+CS
+Wire Wire Line
+	8000 5100 8000 5050
+Wire Wire Line
+	3500 2300 3500 2250
+Wire Wire Line
+	3500 2300 3450 2300
+Wire Wire Line
+	3450 5950 3500 5950
+Wire Wire Line
+	3450 5350 3500 5350
+Connection ~ 3500 5350
+Wire Wire Line
+	3450 4750 3500 4750
+Connection ~ 3500 4750
+Wire Wire Line
+	3450 4150 3500 4150
+Connection ~ 3500 4150
+Wire Wire Line
+	3450 3550 3500 3550
+Wire Wire Line
+	3450 2950 3500 2950
+$Comp
+L power:+24V #PWR?
+U 1 1 622C9690
+P 3500 2250
+F 0 "#PWR?" H 3500 2100 50  0001 C CNN
+F 1 "+24V" H 3515 2423 50  0000 C CNN
+F 2 "" H 3500 2250 50  0001 C CNN
+F 3 "" H 3500 2250 50  0001 C CNN
+	1    3500 2250
+	1    0    0    -1
+$EndComp
 $Comp
 L Connector:Conn_01x01_Female J?
@@
 	-1   0    0    -1
 $EndComp
-Text Label 6700 2900 0    50   ~ 0
-CS
-Text Label 6700 2800 0    50   ~ 0
-SCK
-Text Label 6700 2700 0    50   ~ 0
-MISO
-Text Label 6700 2600 0    50   ~ 0
-MOSI
-Wire Wire Line
-	6900 2600 6650 2600
-Wire Wire Line
-	6650 2700 6900 2700
-Wire Wire Line
-	6650 2800 6900 2800
-Wire Wire Line
-	6650 2900 6900 2900
-Wire Wire Line
-	7550 4850 7700 4850
-Connection ~ 7550 4850
-Wire Wire Line
-	7550 4800 7550 4850
-Wire Wire Line
-	7700 4850 8000 4850
-Connection ~ 7700 4850
-Wire Wire Line
-	7400 4850 7550 4850
-Connection ~ 7400 4850
-Wire Wire Line
-	7100 4850 7400 4850
-$Comp
-L Device:R_Small R?
-U 1 1 61D19CAB
-P 8000 4950
-F 0 "R?" H 8059 4996 50  0000 L CNN
-F 1 "2.2k" H 8059 4905 50  0000 L CNN
-F 2 "" H 8000 4950 50  0001 C CNN
-F 3 "~" H 8000 4950 50  0001 C CNN
-	1    8000 4950
-	-1   0    0    1
-$EndComp
-$Comp
-L Device:R_Small R?
-U 1 1 61D14087
-P 7700 4950
-F 0 "R?" H 7759 4996 50  0000 L CNN
-F 1 "2.2k" H 7759 4905 50  0000 L CNN
-F 2 "" H 7700 4950 50  0001 C CNN
-F 3 "~" H 7700 4950 50  0001 C CNN
-	1    7700 4950
-	-1   0    0    1
-$EndComp
-$Comp
-L Device:R_Small R?
-U 1 1 61D0E598
-P 7400 4950
-F 0 "R?" H 7459 4996 50  0000 L CNN
-F 1 "2.2k" H 7459 4905 50  0000 L CNN
-F 2 "" H 7400 4950 50  0001 C CNN
-F 3 "~" H 7400 4950 50  0001 C CNN
-	1    7400 4950
-	-1   0    0    1
-$EndComp
-$Comp
-L Device:R_Small R?
-U 1 1 61D0640A
-P 7100 4950
-F 0 "R?" H 7159 4996 50  0000 L CNN
-F 1 "2.2k" H 7159 4905 50  0000 L CNN
-F 2 "" H 7100 4950 50  0001 C CNN
-F 3 "~" H 7100 4950 50  0001 C CNN
-	1    7100 4950
-	-1   0    0    1
-$EndComp
-$Comp
-L power:+3.3V #PWR?
-U 1 1 61CFD8CD
-P 7550 4800
-F 0 "#PWR?" H 7550 4650 50  0001 C CNN
-F 1 "+3.3V" H 7565 4973 50  0000 C CNN
-F 2 "" H 7550 4800 50  0001 C CNN
-F 3 "" H 7550 4800 50  0001 C CNN
-	1    7550 4800
-	1    0    0    -1
-$EndComp
-Text Label 7100 5100 3    50   ~ 0
-MOSI
-Wire Wire Line
-	7100 5050 7100 5100
-Text Label 7400 5100 3    50   ~ 0
-MISO
-Wire Wire Line
-	7400 5050 7400 5100
-Text Label 7700 5100 3    50   ~ 0
-SCK
-Wire Wire Line
-	7700 5050 7700 5100
-Text Label 8000 5100 3    50   ~ 0
-CS
-Wire Wire Line
-	8000 5100 8000 5050
-Wire Wire Line
-	3500 2300 3500 2250
-Wire Wire Line
-	3500 2300 3450 2300
-Wire Wire Line
-	3450 5950 3500 5950
-Wire Wire Line
-	3450 5350 3500 5350
-Connection ~ 3500 5350
-Wire Wire Line
-	3450 4750 3500 4750
-Connection ~ 3500 4750
-Wire Wire Line
-	3450 4150 3500 4150
-Connection ~ 3500 4150
-Wire Wire Line
-	3450 3550 3500 3550
-Wire Wire Line
-	3450 2950 3500 2950
-$Comp
-L power:+24V #PWR?
-U 1 1 622C9690
-P 3500 2250
-F 0 "#PWR?" H 3500 2100 50  0001 C CNN
-F 1 "+24V" H 3515 2423 50  0000 C CNN
-F 2 "" H 3500 2250 50  0001 C CNN
-F 3 "" H 3500 2250 50  0001 C CNN
-	1    3500 2250
-	1    0    0    -1
-$EndComp
 $EndSCHEMATC

Commit message: Electrical Rules Checker fixes
Parts:
- BT1: renamed from BT?; footprint (none) -> Connector_PinHeader_2.54mm:PinHeader_1x01_P2.54mm_Vertical
- gave numbers to parts that had none: 31
Connections:
- wire segments 159 -> 164
- no-connect marks 7 -> 8

Commit message: Most of the footprints added
Parts:
- removed Q1: Q_NPN_ECB, symbol Device:Q_NPN_ECB
- added Q1: BC846, Package_TO_SOT_SMD:SOT-23, symbol Transistor_BJT:BC846
- C13, C14, C15, C16, C17: footprint (none) -> Capacitor_SMD:C_0603_1608Metric
- C18: value 0.1uF -> 100nF; footprint (none) -> Capacitor_SMD:C_0603_1608Metric
- J10, J4, J5, J6, J7, J8, J9: footprint (none) -> Connector_PinHeader_2.54mm:PinHeader_1x01_P2.54mm_Vertical
- LTC68101: value LTC6810-1 -> LTC6810-2; footprint (none) -> footprints:LTC6810
- R10, R11, R12, R13, R14, R15, R16, R17, R18, R19, R20: footprint (none) -> Resistor_SMD:R_0603_1608Metric
Changed lines of the file:
@@
 F 0 "C13" H 4742 1946 50  0000 L CNN
 F 1 "1uF" H 4742 1855 50  0000 L CNN
-F 2 "" H 4650 1900 50  0001 C CNN
+F 2 "Capacitor_SMD:C_0603_1608Metric" H 4650 1900 50  0001 C CNN
 F 3 "~" H 4650 1900 50  0001 C CNN
 	1    4650 1900
@@
 F 0 "R10" V 4154 1800 50  0000 C CNN
 F 1 "100" V 4245 1800 50  0000 C CNN
-F 2 "" H 4350 1800 50  0001 C CNN
+F 2 "Resistor_SMD:R_0603_1608Metric" H 4350 1800 50  0001 C CNN
 F 3 "~" H 4350 1800 50  0001 C CNN
 	1    4350 1800
@@
 F 0 "R11" V 4154 2300 50  0000 C CNN
 F 1 "100" V 4245 2300 50  0000 C CNN
-F 2 "" H 4350 2300 50  0001 C CNN
+F 2 "Resistor_SMD:R_0603_1608Metric" H 4350 2300 50  0001 C CNN
 F 3 "~" H 4350 2300 50  0001 C CNN
 	1    4350 2300
@@
 F 0 "C14" H 4742 2446 50  0000 L CNN
 F 1 "10nF" H 4742 2355 50  0000 L CNN
-F 2 "" H 4650 2400 50  0001 C CNN
+F 2 "Capacitor_SMD:C_0603_1608Metric" H 4650 2400 50  0001 C CNN
 F 3 "~" H 4650 2400 50  0001 C CNN
 	1    4650 2400
@@
 F 0 "R12" V 6950 2850 50  0000 C CNN
 F 1 "10k" V 7050 2850 50  0000 C CNN
-F 2 "" H 7000 3000 50  0001 C CNN
+F 2 "Resistor_SMD:R_0603_1608Metric" H 7000 3000 50  0001 C CNN
 F 3 "~" H 7000 3000 50  0001 C CNN
 	1    7000 3000
@@
 F 0 "R13" V 6950 3250 50  0000 C CNN
 F 1 "10k" V 7050 3250 50  0000 C CNN
-F 2 "" H 7000 3100 50  0001 C CNN
+F 2 "Resistor_SMD:R_0603_1608Metric" H 7000 3100 50  0001 C CNN
 F 3 "~" H 7000 3100 50  0001 C CNN
 	1    7000 3100
@@
 F 0 "R14" V 6950 3050 50  0000 C CNN
 F 1 "10k" V 7050 3050 50  0000 C CNN
-F 2 "" H 7000 3200 50  0001 C CNN
+F 2 "Resistor_SMD:R_0603_1608Metric" H 7000 3200 50  0001 C CNN
 F 3 "~" H 7000 3200 50  0001 C CNN
 	1    7000 3200
@@
 F 0 "R15" V 6950 3450 50  0000 C CNN
 F 1 "10k" V 7050 3450 50  0000 C CNN
-F 2 "" H 7000 3300 50  0001 C CNN
+F 2 "Resistor_SMD:R_0603_1608Metric" H 7000 3300 50  0001 C CNN
 F 3 "~" H 7000 3300 50  0001 C CNN
 	1    7000 3300
@@
 F 0 "C15" H 6992 3846 50  0000 L CNN
 F 1 "1uF" H 6992 3755 50  0000 L CNN
-F 2 "" H 6900 3800 50  0001 C CNN
+F 2 "Capacitor_SMD:C_0603_1608Metric" H 6900 3800 50  0001 C CNN
 F 3 "~" H 6900 3800 50  0001 C CNN
 	1    6900 3800
@@
 F 0 "C16" H 7292 3846 50  0000 L CNN
 F 1 "1uF" H 7292 3755 50  0000 L CNN
-F 2 "" H 7200 3800 50  0001 C CNN
+F 2 "Capacitor_SMD:C_0603_1608Metric" H 7200 3800 50  0001 C CNN
 F 3 "~" H 7200 3800 50  0001 C CNN
 	1    7200 3800
@@
 F 0 "C17" H 7592 3846 50  0000 L CNN
 F 1 "1uF" H 7592 3755 50  0000 L CNN
-F 2 "" H 7500 3800 50  0001 C CNN
+F 2 "Capacitor_SMD:C_0603_1608Metric" H 7500 3800 50  0001 C CNN
 F 3 "~" H 7500 3800 50  0001 C CNN
 	1    7500 3800
@@
 P 8100 3150
 F 0 "C18" V 7871 3150 50  0000 C CNN
-F 1 "0.1uF" V 7962 3150 50  0000 C CNN
-F 2 "" H 8100 3150 50  0001 C CNN
+F 1 "100nF" V 7962 3150 50  0000 C CNN
+F 2 "Capacitor_SMD:C_0603_1608Metric" H 8100 3150 50  0001 C CNN
 F 3 "~" H 8100 3150 50  0001 C CNN
 	1    8100 3150
@@
 F 0 "R19" H 7792 2704 50  0000 R CNN
 F 1 "100" H 7792 2795 50  0000 R CNN
-F 2 "" H 7850 2750 50  0001 C CNN
+F 2 "Resistor_SMD:R_0603_1608Metric" H 7850 2750 50  0001 C CNN
 F 3 "~" H 7850 2750 50  0001 C CNN
 	1    7850 2750
@@
 P 6950 4600
 F 0 "LTC68101" H 6050 6965 50  0000 C CNN
-F 1 "LTC6810-1" H 6050 6874 50  0000 C CNN
-F 2 "" H 5800 5650 50  0001 C CNN
+F 1 "LTC6810-2" H 6050 6874 50  0000 C CNN
+F 2 "footprints:LTC6810" H 5800 5650 50  0001 C CNN
 F 3 "" H 5800 5650 50  0001 C CNN
 	1    6950 4600
@@
 Wire Wire Line
 	6650 3400 7550 3400
-$Comp
-L Device:Q_NPN_ECB Q1
-U 1 1 61C0A8C0
-P 7750 3400
-F 0 "Q1" H 7941 3446 50  0000 L CNN
-F 1 "Q_NPN_ECB" H 7941 3355 50  0000 L CNN
-F 2 "" H 7950 3500 50  0001 C CNN
-F 3 "~" H 7750 3400 50  0001 C CNN
-	1    7750 3400
-	1    0    0    -1
-$EndComp
 Wire Wire Line
 	7500 3500 7500 3600
@@
 F 0 "R20" H 8059 4996 50  0000 L CNN
 F 1 "2.2k" H 8059 4905 50  0000 L CNN
-F 2 "" H 8000 4950 50  0001 C CNN
+F 2 "Resistor_SMD:R_0603_1608Metric" H 8000 4950 50  0001 C CNN
 F 3 "~" H 8000 4950 50  0001 C CNN
 	1    8000 4950
@@
 F 0 "R18" H 7759 4996 50  0000 L CNN
 F 1 "2.2k" H 7759 4905 50  0000 L CNN
-F 2 "" H 7700 4950 50  0001 C CNN
+F 2 "Resistor_SMD:R_0603_1608Metric" H 7700 4950 50  0001 C CNN
 F 3 "~" H 7700 4950 50  0001 C CNN
 	1    7700 4950
@@
 F 0 "R17" H 7459 4996 50  0000 L CNN
 F 1 "2.2k" H 7459 4905 50  0000 L CNN
-F 2 "" H 7400 4950 50  0001 C CNN
+F 2 "Resistor_SMD:R_0603_1608Metric" H 7400 4950 50  0001 C CNN
 F 3 "~" H 7400 4950 50  0001 C CNN
 	1    7400 4950
@@
 F 0 "R16" H 7159 4996 50  0000 L CNN
 F 1 "2.2k" H 7159 4905 50  0000 L CNN
-F 2 "" H 7100 4950 50  0001 C CNN
+F 2 "Resistor_SMD:R_0603_1608Metric" H 7100 4950 50  0001 C CNN
 F 3 "~" H 7100 4950 50  0001 C CNN
 	1    7100 4950
@@
 F 0 "J4" H 3650 2400 50  0000 C CNN
 F 1 "Conn_01x01_Female" H 3650 2300 50  0000 C CNN
-F 2 "" H 3250 2300 50  0001 C CNN
+F 2 "Connector_PinHeader_2.54mm:PinHeader_1x01_P2.54mm_Vertical" H 3250 2300 50  0001 C CNN
 F 3 "~" H 3250 2300 50  0001 C CNN
 	1    3250 2300
@@
 F 0 "J5" H 3650 3050 50  0000 C CNN
 F 1 "Conn_01x01_Female" H 3650 2950 50  0000 C CNN
-F 2 "" H 3250 2950 50  0001 C CNN
+F 2 "Connector_PinHeader_2.54mm:PinHeader_1x01_P2.54mm_Vertical" H 3250 2950 50  0001 C CNN
 F 3 "~" H 3250 2950 50  0001 C CNN
 	1    3250 2950
@@
 F 0 "J6" H 3650 3650 50  0000 C CNN
 F 1 "Conn_01x01_Female" H 3650 3550 50  0000 C CNN
-F 2 "" H 3250 3550 50  0001 C CNN
+F 2 "Connector_PinHeader_2.54mm:PinHeader_1x01_P2.54mm_Vertical" H 3250 3550 50  0001 C CNN
 F 3 "~" H 3250 3550 50  0001 C CNN
 	1    3250 3550
@@
 F 0 "J7" H 3650 4250 50  0000 C CNN
 F 1 "Conn_01x01_Female" H 3650 4150 50  0000 C CNN
-F 2 "" H 3250 4150 50  0001 C CNN
+F 2 "Connector_PinHeader_2.54mm:PinHeader_1x01_P2.54mm_Vertical" H 3250 4150 50  0001 C CNN
 F 3 "~" H 3250 4150 50  0001 C CNN
 	1    3250 4150
@@
 F 0 "J8" H 3650 4850 50  0000 C CNN
 F 1 "Conn_01x01_Female" H 3650 4750 50  0000 C CNN
-F 2 "" H 3250 4750 50  0001 C CNN
+F 2 "Connector_PinHeader_2.54mm:PinHeader_1x01_P2.54mm_Vertical" H 3250 4750 50  0001 C CNN
 F 3 "~" H 3250 4750 50  0001 C CNN
 	1    3250 4750
@@
 F 0 "J9" H 3650 5450 50  0000 C CNN
 F 1 "Conn_01x01_Female" H 3650 5350 50  0000 C CNN
-F 2 "" H 3250 5350 50  0001 C CNN
+F 2 "Connector_PinHeader_2.54mm:PinHeader_1x01_P2.54mm_Vertical" H 3250 5350 50  0001 C CNN
 F 3 "~" H 3250 5350 50  0001 C CNN
 	1    3250 5350
@@
 F 0 "J10" H 3650 6050 50  0000 C CNN
 F 1 "Conn_01x01_Female" H 3650 5950 50  0000 C CNN
-F 2 "" H 3250 5950 50  0001 C CNN
+F 2 "Connector_PinHeader_2.54mm:PinHeader_1x01_P2.54mm_Vertical" H 3250 5950 50  0001 C CNN
 F 3 "~" H 3250 5950 50  0001 C CNN
 	1    3250 5950
@@
 Wire Wire Line
 	3500 2100 3500 2300
+$Comp
+L Transistor_BJT:BC846 Q1
+U 1 1 61C11D6C
+P 7750 3400
+F 0 "Q1" H 7941 3446 50  0000 L CNN
+F 1 "BC846" H 7941 3355 50  0000 L CNN
+F 2 "Package_TO_SOT_SMD:SOT-23" H 7950 3325 50  0001 L CIN
+F 3 "https://assets.nexperia.com/documents/data-sheet/BC846_SER.pdf" H 7750 3400 50  0001 L CNN
+	1    7750 3400
+	1    0    0    -1
+$EndComp
 $EndSCHEMATC
