File: HARDWARE/BMS_LV_2022/LTC6810.sch (KiCad schematic (older format))
At the start: 26 parts, among them J11 Conn_01x07_Female, Q1 BC846

Commit message: PCB Layout Update 3
Parts:
- removed R13, R14, R15: 10k, Resistor_SMD:R_0603_1608Metric, symbol Device:R_Small
- added R63: 0, symbol Device:R_Small
Connections:
- net labels added: +BATT, GNDPWR
- net labels removed: +24V
- wire segments 171 -> 173
Other:
- moved on the sheet: R12
Changed lines of the file:
@@
 Comment4 ""
 $EndDescr
-$Sheet
-S 3850 2750 800  400
-U 6199D637
-F0 "Balance1" 50
-F1 "Balance.sch" 50
-F2 "Sx" I R 4650 3000 50
-F3 "Cell" I L 3850 2950 50
-F4 "PreviousBalance" I L 3850 2800 50
-F5 "Cx" I R 4650 2900 50
-F6 "NextBalance" I L 3850 3100 50
-$EndSheet
 Wire Wire Line
 	5450 2600 5350 2600
@@
 	0    1    1    0
 $EndComp
-$Comp
-L power:GND #PWR025
-U 1 1 619FF82A
-P 4650 2000
-F 0 "#PWR025" H 4650 1750 50  0001 C CNN
-F 1 "GND" H 4655 1827 50  0000 C CNN
-F 2 "" H 4650 2000 50  0001 C CNN
-F 3 "" H 4650 2000 50  0001 C CNN
-	1    4650 2000
-	1    0    0    -1
-$EndComp
 Wire Wire Line
 	4250 1800 4000 1800
@@
 F 3 "~" H 4650 2400 50  0001 C CNN
 	1    4650 2400
-	1    0    0    -1
-$EndComp
-$Comp
-L power:GND #PWR026
-U 1 1 61A0AA9E
-P 4650 2500
-F 0 "#PWR026" H 4650 2250 50  0001 C CNN
-F 1 "GND" H 4655 2327 50  0000 C CNN
-F 2 "" H 4650 2500 50  0001 C CNN
-F 3 "" H 4650 2500 50  0001 C CNN
-	1    4650 2500
 	1    0    0    -1
 $EndComp
@@
 L Device:R_Small R12
 U 1 1 61AF3C75
-P 7000 3000
-F 0 "R12" V 6950 2850 50  0000 C CNN
-F 1 "10k" V 7050 2850 50  0000 C CNN
-F 2 "Resistor_SMD:R_0603_1608Metric" H 7000 3000 50  0001 C CNN
-F 3 "~" H 7000 3000 50  0001 C CNN
-	1    7000 3000
-	0    1    1    0
-$EndComp
-$Comp
-L Device:R_Small R13
-U 1 1 61AF526B
-P 7000 3100
-F 0 "R13" V 6950 3250 50  0000 C CNN
-F 1 "10k" V 7050 3250 50  0000 C CNN
-F 2 "Resistor_SMD:R_0603_1608Metric" H 7000 3100 50  0001 C CNN
-F 3 "~" H 7000 3100 50  0001 C CNN
-	1    7000 3100
+P 7050 3150
+F 0 "R12" V 6950 3150 50  0000 C CNN
+F 1 "10k" V 7150 3150 50  0000 C CNN
+F 2 "Resistor_SMD:R_0603_1608Metric" H 7050 3150 50  0001 C CNN
+F 3 "~" H 7050 3150 50  0001 C CNN
+	1    7050 3150
 	0    1    1    0
 $EndComp
@@
 Text HLabel 6900 2900 2    50   Input ~ 0
 CS
-$Comp
-L Device:R_Small R14
-U 1 1 61B17B8B
-P 7000 3200
-F 0 "R14" V 6950 3050 50  0000 C CNN
-F 1 "10k" V 7050 3050 50  0000 C CNN
-F 2 "Resistor_SMD:R_0603_1608Metric" H 7000 3200 50  0001 C CNN
-F 3 "~" H 7000 3200 50  0001 C CNN
-	1    7000 3200
-	0    1    1    0
-$EndComp
-$Comp
-L Device:R_Small R15
-U 1 1 61B17B91
-P 7000 3300
-F 0 "R15" V 6950 3450 50  0000 C CNN
-F 1 "10k" V 7050 3450 50  0000 C CNN
-F 2 "Resistor_SMD:R_0603_1608Metric" H 7000 3300 50  0001 C CNN
-F 3 "~" H 7000 3300 50  0001 C CNN
-	1    7000 3300
-	0    1    1    0
-$EndComp
 Wire Wire Line
 	6650 3700 6900 3700
@@
 F 3 "~" H 7500 3800 50  0001 C CNN
 	1    7500 3800
-	1    0    0    -1
-$EndComp
-$Comp
-L power:GND #PWR028
-U 1 1 61B88F45
-P 7200 3950
-F 0 "#PWR028" H 7200 3700 50  0001 C CNN
-F 1 "GND" H 7205 3777 50  0000 C CNN
-F 2 "" H 7200 3950 50  0001 C CNN
-F 3 "" H 7200 3950 50  0001 C CNN
-	1    7200 3950
 	1    0    0    -1
 $EndComp
@@
 	6650 3000 6900 3000
 $Comp
-L power:GND #PWR031
-U 1 1 61CD490A
-P 8350 3150
-F 0 "#PWR031" H 8350 2900 50  0001 C CNN
-F 1 "GND" H 8355 2977 50  0000 C CNN
-F 2 "" H 8350 3150 50  0001 C CNN
-F 3 "" H 8350 3150 50  0001 C CNN
-	1    8350 3150
-	1    0    0    -1
-$EndComp
-$Comp
 L BMS_LV_2022-rescue:LTC6810-1-LTC6810-1 LTC68101
 U 1 1 61D92574
@@
 $EndComp
 Wire Wire Line
-	7100 3200 7250 3200
-Wire Wire Line
-	7250 3100 7100 3100
-Wire Wire Line
-	7250 3100 7250 3000
-Wire Wire Line
-	7250 3000 7100 3000
-Connection ~ 7250 3100
-Wire Wire Line
-	7250 3200 7250 3300
-Wire Wire Line
-	7250 3300 7100 3300
-Connection ~ 7250 3200
-Wire Wire Line
-	7250 3200 7250 3100
-Wire Wire Line
-	7250 3100 7350 3100
-$Comp
-L power:GND #PWR029
-U 1 1 61E1873A
-P 7350 3100
-F 0 "#PWR029" H 7350 2850 50  0001 C CNN
-F 1 "GND" H 7355 2927 50  0000 C CNN
-F 2 "" H 7350 3100 50  0001 C CNN
-F 3 "" H 7350 3100 50  0001 C CNN
-	1    7350 3100
-	1    0    0    -1
-$EndComp
-Wire Wire Line
 	6650 3400 7550 3400
 Wire Wire Line
@@
 	5400 4800 5650 4800
 Connection ~ 5650 4800
-$Comp
-L power:GND #PWR027
-U 1 1 61EBBC18
-P 6050 4900
-F 0 "#PWR027" H 6050 4650 50  0001 C CNN
-F 1 "GND" H 6055 4727 50  0000 C CNN
-F 2 "" H 6050 4900 50  0001 C CNN
-F 3 "" H 6050 4900 50  0001 C CNN
-	1    6050 4900
-	1    0    0    -1
-$EndComp
 Wire Wire Line
 	6050 4800 6050 4900
@@
 Connection ~ 3500 4750
 Connection ~ 3500 4150
-$Comp
-L power:+24V #PWR015
-U 1 1 622C9690
-P 3500 2050
-F 0 "#PWR015" H 3500 1900 50  0001 C CNN
-F 1 "+24V" H 3515 2223 50  0000 C CNN
-F 2 "" H 3500 2050 50  0001 C CNN
-F 3 "" H 3500 2050 50  0001 C CNN
-	1    3500 2050
-	1    0    0    -1
-$EndComp
 NoConn ~ 5450 2500
 $Comp
@@
 L power:GND #PWR024
 U 1 1 61AB7502
-P 3500 6000
-F 0 "#PWR024" H 3500 5750 50  0001 C CNN
-F 1 "GND" H 3505 5827 50  0000 C CNN
-F 2 "" H 3500 6000 50  0001 C CNN
-F 3 "" H 3500 6000 50  0001 C CNN
-	1    3500 6000
+P 4500 6700
+F 0 "#PWR024" H 4500 6450 50  0001 C CNN
+F 1 "GND" H 4505 6527 50  0000 C CNN
+F 2 "" H 4500 6700 50  0001 C CNN
+F 3 "" H 4500 6700 50  0001 C CNN
+	1    4500 6700
 	1    0    0    -1
 $EndComp
@@
 Wire Wire Line
 	2050 4050 1950 4050
+$Comp
+L power:GNDPWR #PWR0104
+U 1 1 61EA8090
+P 3500 6000
+F 0 "#PWR0104" H 3500 5800 50  0001 C CNN
+F 1 "GNDPWR" H 3504 5846 50  0000 C CNN
+F 2 "" H 3500 5950 50  0001 C CNN
+F 3 "" H 3500 5950 50  0001 C CNN
+	1    3500 6000
+	1    0    0    -1
+$EndComp
+$Comp
+L power:GNDPWR #PWR0105
+U 1 1 61EBD8BF
+P 4100 6700
+F 0 "#PWR0105" H 4100 6500 50  0001 C CNN
+F 1 "GNDPWR" H 4104 6546 50  0000 C CNN
+F 2 "" H 4100 6650 50  0001 C CNN
+F 3 "" H 4100 6650 50  0001 C CNN
+	1    4100 6700
+	1    0    0    -1
+$EndComp
+$Comp
+L Device:R_Small R63
+U 1 1 61ECEFC7
+P 4300 6700
+F 0 "R63" V 4104 6700 50  0000 C CNN
+F 1 "0" V 4195 6700 50  0000 C CNN
+F 2 "" H 4300 6700 50  0001 C CNN
+F 3 "~" H 4300 6700 50  0001 C CNN
+	1    4300 6700
+	0    1    1    0
+$EndComp
+Wire Wire Line
+	4100 6700 4200 6700
+Wire Wire Line
+	4400 6700 4500 6700
+$Comp
+L power:GNDPWR #PWR0106
+U 1 1 61EEC608
+P 6050 4900
+F 0 "#PWR0106" H 6050 4700 50  0001 C CNN
+F 1 "GNDPWR" H 6054 4746 50  0000 C CNN
+F 2 "" H 6050 4850 50  0001 C CNN
+F 3 "" H 6050 4850 50  0001 C CNN
+	1    6050 4900
+	1    0    0    -1
+$EndComp
+$Comp
+L power:GNDPWR #PWR0108
+U 1 1 61F37B6B
+P 4650 2050
+F 0 "#PWR0108" H 4650 1850 50  0001 C CNN
+F 1 "GNDPWR" H 4654 1896 50  0000 C CNN
+F 2 "" H 4650 2000 50  0001 C CNN
+F 3 "" H 4650 2000 50  0001 C CNN
+	1    4650 2050
+	1    0    0    -1
+$EndComp
+Wire Wire Line
+	4650 2500 4650 2550
+Wire Wire Line
+	4650 2050 4650 2000
+$Comp
+L power:GNDPWR #PWR0109
+U 1 1 61F775E3
+P 8350 3150
+F 0 "#PWR0109" H 8350 2950 50  0001 C CNN
+F 1 "GNDPWR" H 8354 2996 50  0000 C CNN
+F 2 "" H 8350 3100 50  0001 C CNN
+F 3 "" H 8350 3100 50  0001 C CNN
+	1    8350 3150
+	1    0    0    -1
+$EndComp
+$Comp
+L power:GNDPWR #PWR0110
+U 1 1 61F80785
+P 7200 3950
+F 0 "#PWR0110" H 7200 3750 50  0001 C CNN
+F 1 "GNDPWR" H 7204 3796 50  0000 C CNN
+F 2 "" H 7200 3900 50  0001 C CNN
+F 3 "" H 7200 3900 50  0001 C CNN
+	1    7200 3950
+	1    0    0    -1
+$EndComp
+$Comp
+L power:GNDPWR #PWR0111
+U 1 1 61F9C6CA
+P 7350 3150
+F 0 "#PWR0111" H 7350 2950 50  0001 C CNN
+F 1 "GNDPWR" H 7354 2996 50  0000 C CNN
+F 2 "" H 7350 3100 50  0001 C CNN
+F 3 "" H 7350 3100 50  0001 C CNN
+	1    7350 3150
+	1    0    0    -1
+$EndComp
+Wire Wire Line
+	6900 3000 6900 3100
+Connection ~ 6900 3100
+Wire Wire Line
+	6900 3100 6900 3150
+Connection ~ 6900 3200
+Wire Wire Line
+	6900 3200 6900 3300
+Wire Wire Line
+	6900 3150 6950 3150
+Connection ~ 6900 3150
+Wire Wire Line
+	6900 3150 6900 3200
+Wire Wire Line
+	7150 3150 7350 3150
+$Comp
+L power:GNDPWR #PWR0107
+U 1 1 61F2EC75
+P 4650 2550
+F 0 "#PWR0107" H 4650 2350 50  0001 C CNN
+F 1 "GNDPWR" H 4654 2396 50  0000 C CNN
+F 2 "" H 4650 2500 50  0001 C CNN
+F 3 "" H 4650 2500 50  0001 C CNN
+	1    4650 2550
+	1    0    0    -1
+$EndComp
+$Sheet
+S 3850 2750 800  400
+U 6199D637
+F0 "Balance1" 50
+F1 "Balance.sch" 50
+F2 "Sx" I R 4650 3000 50
+F3 "Cell" I L 3850 2950 50
+F4 "PreviousBalance" I L 3850 2800 50
+F5 "Cx" I R 4650 2900 50
+F6 "NextBalance" I L 3850 3100 50
+$EndSheet
+$Comp
+L power:+BATT #PWR0120
+U 1 1 61F3FA17
+P 3500 2050
+F 0 "#PWR0120" H 3500 1900 50  0001 C CNN
+F 1 "+BATT" H 3515 2223 50  0000 C CNN
+F 2 "" H 3500 2050 50  0001 C CNN
+F 3 "" H 3500 2050 50  0001 C CNN
+	1    3500 2050
+	1    0    0    -1
+$EndComp
 $EndSCHEMATC

Commit message: Power planes added
Parts:
- Q1: symbol Transistor_BJT:BC846 -> BMS_LV_2022-rescue:BC846-Transistor_BJT
Changed lines of the file:
@@
 EESchema Schematic File Version 4
-EELAYER 30 0
+LIBS:BMS_LV_2022-cache
+EELAYER 29 0
 EELAYER END
 $Descr A4 11693 8268
@@
 	3500 2100 3500 2300
 $Comp
-L Transistor_BJT:BC846 Q1
+L BMS_LV_2022-rescue:BC846-Transistor_BJT Q1
 U 1 1 61C11D6C
 P 7750 3400
+AR Path="/61C11D6C" Ref="Q1"  Part="1"
+AR Path="/61996AA1/61C11D6C" Ref="Q1"  Part="1"
 F 0 "Q1" H 7941 3446 50  0000 L CNN
 F 1 "BC846" H 7941 3355 50  0000 L CNN

Commit message: PCB Routing Update 2
Parts:
- LTC68101: symbol BMS_LV_2022-rescue:LTC6810-1-LTC6810-1 -> ltc6810-2:LTC6810-2
Changed lines of the file:
@@
 	6650 3000 6900 3000
 $Comp
-L BMS_LV_2022-rescue:LTC6810-1-LTC6810-1 LTC68101
+L ltc6810-2:LTC6810-2 LTC68101
 U 1 1 61D92574
 P 6950 4600

Commit message: HARDWARE Release V1.0
Parts:
- removed R63: 0, symbol Device:R_Small
Connections:
- wire segments 173 -> 172
Changed lines of the file:
@@
 $EndComp
-$Comp
-L Device:R_Small R63
-U 1 1 61ECEFC7
-P 4300 6700
-F 0 "R63" V 4104 6700 50  0000 C CNN
-F 1 "0" V 4195 6700 50  0000 C CNN
-F 2 "" H 4300 6700 50  0001 C CNN
-F 3 "~" H 4300 6700 50  0001 C CNN
-	1    4300 6700
-	0    1    1    0
-$EndComp
-Wire Wire Line
-	4100 6700 4200 6700
-Wire Wire Line
-	4400 6700 4500 6700
 $Comp
 L power:GNDPWR #PWR0106
@@
 	1    0    0    -1
 $EndComp
+Wire Wire Line
+	4100 6700 4500 6700
 $EndSCHEMATC
