File: HARDWARE/BMS_LV_2022/BMS_LV_2022.sch (KiCad schematic (older format))
At the start: 28 parts, among them J1 Conn_01x06_Male, J2 Conn_01x12_Male, J3 USB_B_Mini, SW1 SW_Push, U1 STM32L4P5RET6, Y1 Crystal

Commit message: PCB Layout Update 3
Parts:
- removed Y1: Crystal, Crystal:Crystal_SMD_3225-4Pin_3.2x2.5mm, symbol Device:Crystal
- added J4: Battery+, footprints:CellPad, symbol Connector:Conn_01x01_Male
- added J5: Battery-, footprints:CellPad, symbol Connector:Conn_01x01_Male
- added Y1: Crystal, Crystal:Crystal_SMD_3225-4Pin_3.2x2.5mm, symbol Device:Crystal_GND24_Small
Connections:
- net GND: now also J5.1 (Pin_1), Y1.2, Y1.4
- net VCC: now also J2.6 (Pin_6); no longer J2.8 (Pin_8)
- net at C5.2, U1.5 (PH0-OSC_IN): now also Y1.3
- net at C6.2, U1.6 (PH1-OSC_OUT): now also Y1.1
- new net +24V: J4.1 (Pin_1)
Other:
- note added: "Main current path"
Changed lines of the file:
@@
 Wire Wire Line
 	1700 5350 1900 5350
-$Comp
-L Device:Crystal Y1
-U 1 1 61F31AAD
-P 5100 3500
-F 0 "Y1" V 5054 3369 50  0000 R CNN
-F 1 "Crystal" V 5145 3369 50  0000 R CNN
-F 2 "Crystal:Crystal_SMD_3225-4Pin_3.2x2.5mm" H 5100 3500 50  0001 C CNN
-F 3 "~" H 5100 3500 50  0001 C CNN
-	1    5100 3500
-	0    -1   1    0
-$EndComp
 Wire Wire Line
 	5550 3300 5550 3450
 Wire Wire Line
 	5550 3550 5550 3700
-Wire Wire Line
-	5100 3700 5100 3650
-Wire Wire Line
-	5100 3300 5100 3350
 $Comp
 L Device:C_Small C6
@@
 Connection ~ 4600 3300
 Wire Wire Line
-	4600 3300 4600 3700
-Wire Wire Line
 	4600 3700 4600 3750
 Connection ~ 4600 3700
@@
 U 1 1 61F57B55
 P 4900 3300
-F 0 "C5" V 4671 3300 50  0000 C CNN
-F 1 "22pF" V 4762 3300 50  0000 C CNN
+F 0 "C5" V 4850 3450 50  0000 C CNN
+F 1 "22pF" V 4950 3450 50  0000 C CNN
 F 2 "Capacitor_SMD:C_0603_1608Metric" H 4900 3300 50  0001 C CNN
 F 3 "~" H 4900 3300 50  0001 C CNN
@@
 Wire Wire Line
 	10500 4550 10450 4550
-Text Notes 9150 4350 0    50   ~ 0
+Text Notes 9200 4250 0    50   ~ 0
 Shorted when \nconnector is connected
 Text Notes 9450 700  0    157  ~ 31
 Connectors
-Wire Notes Line
-	9000 500  9000 5000
 Wire Notes Line
 	9000 5000 11200 5000
@@
 VCC_Pin
 Wire Bus Line
-	10250 4350 10150 4350
+	10250 4250 10150 4250
 Wire Bus Line
-	10150 4350 10150 4250
+	10150 4250 10150 4150
 Wire Bus Line
-	10150 4250 10250 4250
+	10150 4150 10250 4150
 Wire Notes Line
 	10050 4400 11200 4400
@@
 NoConn ~ 6950 5500
 NoConn ~ 6950 5600
-NoConn ~ 10450 4150
+NoConn ~ 10450 4350
 NoConn ~ 10350 1500
 Text Notes 1200 5200 0    118  ~ 0
@@
 	6150 1800 6150 1700
 Wire Wire Line
-	10450 4350 11000 4350
+	10450 4150 11000 4150
 $Comp
 L power:VCC #PWR014
 U 1 1 622C0542
-P 11000 4350
-F 0 "#PWR014" H 11000 4200 50  0001 C CNN
-F 1 "VCC" H 11015 4523 50  0000 C CNN
-F 2 "" H 11000 4350 50  0001 C CNN
-F 3 "" H 11000 4350 50  0001 C CNN
-	1    11000 4350
+P 11000 4150
+F 0 "#PWR014" H 11000 4000 50  0001 C CNN
+F 1 "VCC" H 11015 4323 50  0000 C CNN
+F 2 "" H 11000 4150 50  0001 C CNN
+F 3 "" H 11000 4150 50  0001 C CNN
+	1    11000 4150
 	1    0    0    -1
 $EndComp
@@
 Wire Wire Line
 	10500 4700 10500 4650
+$Comp
+L Device:Crystal_GND24_Small Y1
+U 1 1 61FCA236
+P 5100 3500
+F 0 "Y1" V 5250 3250 50  0000 L CNN
+F 1 "Crystal" V 5200 3150 50  0000 L CNN
+F 2 "Crystal:Crystal_SMD_3225-4Pin_3.2x2.5mm" H 5100 3500 50  0001 C CNN
+F 3 "~" H 5100 3500 50  0001 C CNN
+	1    5100 3500
+	0    -1   -1   0
+$EndComp
+Wire Wire Line
+	5100 3600 5100 3700
+Wire Wire Line
+	5100 3300 5100 3400
+Wire Wire Line
+	4600 3300 4600 3500
+Wire Wire Line
+	5000 3500 4600 3500
+Connection ~ 4600 3500
+Wire Wire Line
+	4600 3500 4600 3700
+$Comp
+L power:GND #PWR0103
+U 1 1 6201D764
+P 5350 3500
+F 0 "#PWR0103" H 5350 3250 50  0001 C CNN
+F 1 "GND" H 5355 3327 50  0000 C CNN
+F 2 "" H 5350 3500 50  0001 C CNN
+F 3 "" H 5350 3500 50  0001 C CNN
+	1    5350 3500
+	1    0    0    -1
+$EndComp
+Wire Wire Line
+	5200 3500 5350 3500
+$Comp
+L Connector:Conn_01x01_Male J4
+U 1 1 61EDCBEE
+P 10050 5350
+F 0 "J4" H 10150 5600 50  0000 C CNN
+F 1 "Battery+" H 10150 5500 50  0000 C CNN
+F 2 "footprints:CellPad" H 10050 5350 50  0001 C CNN
+F 3 "~" H 10050 5350 50  0001 C CNN
+	1    10050 5350
+	1    0    0    -1
+$EndComp
+$Comp
+L Connector:Conn_01x01_Male J5
+U 1 1 61EDDCD4
+P 10050 5700
+F 0 "J5" H 10150 5950 50  0000 C CNN
+F 1 "Battery-" H 10150 5850 50  0000 C CNN
+F 2 "footprints:CellPad" H 10050 5700 50  0001 C CNN
+F 3 "~" H 10050 5700 50  0001 C CNN
+	1    10050 5700
+	1    0    0    -1
+$EndComp
+Wire Wire Line
+	10250 5350 10450 5350
+Wire Wire Line
+	10250 5700 10450 5700
+$Comp
+L power:GND #PWR0118
+U 1 1 61EF3195
+P 10450 5700
+F 0 "#PWR0118" H 10450 5450 50  0001 C CNN
+F 1 "GND" H 10455 5527 50  0000 C CNN
+F 2 "" H 10450 5700 50  0001 C CNN
+F 3 "" H 10450 5700 50  0001 C CNN
+	1    10450 5700
+	1    0    0    -1
+$EndComp
+Wire Notes Line
+	9000 6050 11200 6050
+Wire Notes Line
+	9000 500  9000 6050
+Text Notes 9100 5150 0    59   ~ 12
+Main current path
+$Comp
+L power:+24V #PWR0119
+U 1 1 61F35FDA
+P 10450 5350
+F 0 "#PWR0119" H 10450 5200 50  0001 C CNN
+F 1 "+24V" H 10465 5523 50  0000 C CNN
+F 2 "" H 10450 5350 50  0001 C CNN
+F 3 "" H 10450 5350 50  0001 C CNN
+	1    10450 5350
+	1    0    0    -1
+$EndComp
 $EndSCHEMATC

Commit message: Power planes added
Parts:
- J3: symbol Connector:USB_B_Mini -> BMS_LV_2022-rescue:USB_B_Mini-Connector
Changed lines of the file:
@@
 EESchema Schematic File Version 4
-EELAYER 30 0
+LIBS:BMS_LV_2022-cache
+EELAYER 29 0
 EELAYER END
 $Descr A4 11693 8268
@@
 USB-DP
 $Comp
-L Connector:USB_B_Mini J3
+L BMS_LV_2022-rescue:USB_B_Mini-Connector J3
 U 1 1 62011569
 P 10650 1300
