File: HARDWARE/BMS_LV_2022/eFuse.sch (KiCad schematic (older format))
At the start: 11 parts

Commit message: Hardware update; -changes after team review;
Parts:
- added F?: Polyfuse, symbol Device:Polyfuse
- C?: value C_Small -> 0*
- R?: value R_Small -> 10k
- R?: value R_Small -> 100
Connections:
- net labels added: VCC_Pin
- wire segments 38 -> 41
Changed lines of the file:
@@
 L power:+24V #PWR?
 U 1 1 626B571F
-P 2550 1450
+P 1900 1450
 AR Path="/626B571F" Ref="#PWR?"  Part="1"
 AR Path="/6269845F/626B571F" Ref="#PWR?"  Part="1"
-F 0 "#PWR?" H 2550 1300 50  0001 C CNN
-F 1 "+24V" H 2565 1623 50  0000 C CNN
-F 2 "" H 2550 1450 50  0001 C CNN
-F 3 "" H 2550 1450 50  0001 C CNN
-	1    2550 1450
+F 0 "#PWR?" H 1900 1300 50  0001 C CNN
+F 1 "+24V" H 1915 1623 50  0000 C CNN
+F 2 "" H 1900 1450 50  0001 C CNN
+F 3 "" H 1900 1450 50  0001 C CNN
+	1    1900 1450
 	1    0    0    -1
 $EndComp
@@
 	3500 2000 3600 2000
 Wire Wire Line
-	2750 2000 2750 1450
-Wire Wire Line
 	3600 2000 3600 900
 Connection ~ 3600 2000
 Wire Wire Line
 	3600 2000 3700 2000
-Connection ~ 2750 1450
-Wire Wire Line
-	2750 1450 2750 900
 $Comp
 L Transistor_FET:BSS138 Q?
@@
 P 3500 2200
 F 0 "C?" H 3408 2154 50  0000 R CNN
-F 1 "C_Small" H 3408 2245 50  0000 R CNN
+F 1 "0*" H 3408 2245 50  0000 R CNN
 F 2 "" H 3500 2200 50  0001 C CNN
 F 3 "~" H 3500 2200 50  0001 C CNN
 	1    3500 2200
-	1    0    0    -1
+	1    0    0    1
 $EndComp
 $Comp
@@
 P 3700 2200
 F 0 "R?" H 3759 2246 50  0000 L CNN
-F 1 "R_Small" H 3759 2155 50  0000 L CNN
+F 1 "10k" H 3759 2155 50  0000 L CNN
 F 2 "" H 3700 2200 50  0001 C CNN
 F 3 "~" H 3700 2200 50  0001 C CNN
@@
 Wire Wire Line
 	4450 2000 4400 2000
-Wire Wire Line
-	2550 1450 2750 1450
 $Comp
 L Device:Fuse F?
@@
 F 3 "~" H 4200 1000 50  0001 C CNN
 	1    4200 1000
-	0    -1   -1   0
+	0    1    -1   0
 $EndComp
 Text HLabel 2800 3550 0    50   Input ~ 0
@@
 P 3600 3100
 F 0 "R?" H 3659 3146 50  0000 L CNN
-F 1 "R_Small" H 3659 3055 50  0000 L CNN
+F 1 "100" H 3659 3055 50  0000 L CNN
 F 2 "" H 3600 3100 50  0001 C CNN
 F 3 "~" H 3600 3100 50  0001 C CNN
@@
 Text HLabel 4950 1450 2    50   Output ~ 0
 CurrentSensor_IP+
+Wire Wire Line
+	2750 900  2750 1450
+Connection ~ 2750 1450
+Wire Wire Line
+	2750 1450 2750 2000
+Wire Wire Line
+	2500 1450 2500 1300
+Connection ~ 2500 1450
+Wire Wire Line
+	2500 1450 2750 1450
+Text HLabel 2500 900  1    50   Output ~ 0
+VCC_Pin
+Wire Wire Line
+	2500 1000 2500 900
+$Comp
+L Device:Polyfuse F?
+U 1 1 61C9E38A
+P 2500 1150
+F 0 "F?" H 2588 1196 50  0000 L CNN
+F 1 "Polyfuse" H 2588 1105 50  0000 L CNN
+F 2 "" H 2550 950 50  0001 L CNN
+F 3 "~" H 2500 1150 50  0001 C CNN
+	1    2500 1150
+	-1   0    0    -1
+$EndComp
+Wire Wire Line
+	1900 1450 2500 1450
 $EndSCHEMATC

Commit message: Electrical Rules Checker fixes
Parts:
- gave numbers to parts that had none: 12
Changed lines of the file:
@@
 P 1900 1450
 AR Path="/626B571F" Ref="#PWR?"  Part="1"
-AR Path="/6269845F/626B571F" Ref="#PWR?"  Part="1"
-F 0 "#PWR?" H 1900 1300 50  0001 C CNN
+AR Path="/6269845F/626B571F" Ref="#PWR047"  Part="1"
+F 0 "#PWR047" H 1900 1300 50  0001 C CNN
 F 1 "+24V" H 1915 1623 50  0000 C CNN
 F 2 "" H 1900 1450 50  0001 C CNN
@@
 P 3600 3850
 AR Path="/626B572C" Ref="#PWR?"  Part="1"
-AR Path="/6269845F/626B572C" Ref="#PWR?"  Part="1"
-F 0 "#PWR?" H 3600 3600 50  0001 C CNN
+AR Path="/6269845F/626B572C" Ref="#PWR048"  Part="1"
+F 0 "#PWR048" H 3600 3600 50  0001 C CNN
 F 1 "GND" H 3605 3677 50  0000 C CNN
 F 2 "" H 3600 3850 50  0001 C CNN
@@
 P 3500 3550
 AR Path="/626B577C" Ref="Q?"  Part="1"
-AR Path="/6269845F/626B577C" Ref="Q?"  Part="1"
-F 0 "Q?" H 3704 3596 50  0000 L CNN
+AR Path="/6269845F/626B577C" Ref="Q10"  Part="1"
+F 0 "Q10" H 3704 3596 50  0000 L CNN
 F 1 "BSS138" H 3704 3505 50  0000 L CNN
 F 2 "Package_TO_SOT_SMD:SOT-23" H 3700 3475 50  0001 L CIN
@@
 P 3050 3550
 AR Path="/626B5786" Ref="R?"  Part="1"
-AR Path="/6269845F/626B5786" Ref="R?"  Part="1"
-F 0 "R?" V 2854 3550 50  0000 C CNN
+AR Path="/6269845F/626B5786" Ref="R59"  Part="1"
+F 0 "R59" V 2854 3550 50  0000 C CNN
 F 1 "100" V 2945 3550 50  0000 C CNN
 F 2 "" H 3050 3550 50  0001 C CNN
@@
 P 3350 3800
 AR Path="/626B578C" Ref="R?"  Part="1"
-AR Path="/6269845F/626B578C" Ref="R?"  Part="1"
-F 0 "R?" V 3546 3800 50  0000 C CNN
+AR Path="/6269845F/626B578C" Ref="R60"  Part="1"
+F 0 "R60" V 3546 3800 50  0000 C CNN
 F 1 "10k" V 3455 3800 50  0000 C CNN
 F 2 "" H 3350 3800 50  0001 C CNN
@@
 Connection ~ 3200 3550
 $Comp
-L Device:C_Small C?
+L Device:C_Small C41
 U 1 1 62872278
 P 3500 2200
-F 0 "C?" H 3408 2154 50  0000 R CNN
+F 0 "C41" H 3408 2154 50  0000 R CNN
 F 1 "0*" H 3408 2245 50  0000 R CNN
 F 2 "" H 3500 2200 50  0001 C CNN
@@
 $EndComp
 $Comp
-L Device:R_Small R?
+L Device:R_Small R62
 U 1 1 62874194
 P 3700 2200
-F 0 "R?" H 3759 2246 50  0000 L CNN
+F 0 "R62" H 3759 2246 50  0000 L CNN
 F 1 "10k" H 3759 2155 50  0000 L CNN
 F 2 "" H 3700 2200 50  0001 C CNN
@@
 	4450 2000 4400 2000
 $Comp
-L Device:Fuse F?
+L Device:Fuse F2
 U 1 1 6287D375
 P 4700 1450
-F 0 "F?" V 4503 1450 50  0000 C CNN
+F 0 "F2" V 4503 1450 50  0000 C CNN
 F 1 "Fuse" V 4594 1450 50  0000 C CNN
 F 2 "" V 4630 1450 50  0001 C CNN
@@
 $EndComp
 $Comp
-L Device:Q_PMOS_GDS Q?
+L Device:Q_PMOS_GDS Q9
 U 1 1 6287F1CD
 P 3000 2100
-F 0 "Q?" V 3342 2100 50  0000 C CNN
+F 0 "Q9" V 3342 2100 50  0000 C CNN
 F 1 "Q_PMOS_GDS" V 3251 2100 50  0000 C CNN
 F 2 "" H 3200 2200 50  0001 C CNN
@@
 $EndComp
 $Comp
-L Device:Q_PMOS_GDS Q?
+L Device:Q_PMOS_GDS Q8
 U 1 1 62882C0C
 P 3000 1000
-F 0 "Q?" V 3342 1000 50  0000 C CNN
+F 0 "Q8" V 3342 1000 50  0000 C CNN
 F 1 "Q_PMOS_GDS" V 3251 1000 50  0000 C CNN
 F 2 "" H 3200 1100 50  0001 C CNN
@@
 $EndComp
 $Comp
-L Device:Q_PMOS_GDS Q?
+L Device:Q_PMOS_GDS Q12
 U 1 1 62883BEA
 P 4200 2100
-F 0 "Q?" V 4542 2100 50  0000 C CNN
+F 0 "Q12" V 4542 2100 50  0000 C CNN
 F 1 "Q_PMOS_GDS" V 4451 2100 50  0000 C CNN
 F 2 "" H 4400 2200 50  0001 C CNN
@@
 $EndComp
 $Comp
-L Device:Q_PMOS_GDS Q?
+L Device:Q_PMOS_GDS Q11
 U 1 1 62886B18
 P 4200 1000
-F 0 "Q?" V 4542 1000 50  0000 C CNN
+F 0 "Q11" V 4542 1000 50  0000 C CNN
 F 1 "Q_PMOS_GDS" V 4451 1000 50  0000 C CNN
 F 2 "" H 4400 1100 50  0001 C CNN
@@
 Switch_Signal
 $Comp
-L Device:R_Small R?
+L Device:R_Small R61
 U 1 1 62887CEF
 P 3600 3100
-F 0 "R?" H 3659 3146 50  0000 L CNN
+F 0 "R61" H 3659 3146 50  0000 L CNN
 F 1 "100" H 3659 3055 50  0000 L CNN
 F 2 "" H 3600 3100 50  0001 C CNN
@@
 	2500 1000 2500 900
 $Comp
-L Device:Polyfuse F?
+L Device:Polyfuse F1
 U 1 1 61C9E38A
 P 2500 1150
-F 0 "F?" H 2588 1196 50  0000 L CNN
+F 0 "F1" H 2588 1196 50  0000 L CNN
 F 1 "Polyfuse" H 2588 1105 50  0000 L CNN
 F 2 "" H 2550 950 50  0001 L CNN

Commit message: Most of the footprints added
Parts:
- removed Q11, Q12, Q8, Q9: Q_PMOS_GDS, symbol Device:Q_PMOS_GDS
- added Q11, Q12, Q8, Q9: Q_PMOS_GSD, Package_TO_SOT_SMD:SOT-23, symbol Device:Q_PMOS_GSD
- C41: footprint (none) -> Capacitor_SMD:C_0603_1608Metric
- R59, R60, R61, R62: footprint (none) -> Resistor_SMD:R_0603_1608Metric
Other:
- moved on the sheet: C41, F1, F2, Q10, R59, R60, R61, R62

Commit message: PCB layout init
Parts:
- F1: footprint (none) -> Diode_SMD:D_SMB
- F2: footprint (none) -> Fuse:Fuseholder_Blade_Mini_Keystone_3568
Changed lines of the file:
@@
 F 0 "F2" V 6853 2800 50  0000 C CNN
 F 1 "Fuse" V 6944 2800 50  0000 C CNN
-F 2 "" V 6980 2800 50  0001 C CNN
+F 2 "Fuse:Fuseholder_Blade_Mini_Keystone_3568" V 6980 2800 50  0001 C CNN
 F 3 "~" H 7050 2800 50  0001 C CNN
 	1    7050 2800
@@
 F 0 "F1" H 4938 2546 50  0000 L CNN
 F 1 "Polyfuse" H 4938 2455 50  0000 L CNN
-F 2 "" H 4900 2300 50  0001 L CNN
+F 2 "Diode_SMD:D_SMB" H 4900 2300 50  0001 L CNN
 F 3 "~" H 4850 2500 50  0001 C CNN
 	1    4850 2500

Commit message: PCB update
Parts changed due to smaller footprints
Parts:
- F1: footprint Diode_SMD:D_SMB -> Fuse:Fuse_1206_3216Metric; Part Number (none) -> 0ZCJ0020FF2E
- F2: footprint Fuse:Fuseholder_Blade_Mini_Keystone_3568 -> footprints:Fuseholder_Keystone_3522-2; Part Number (none) -> 3522-2
Changed lines of the file:
@@
 F 0 "F2" V 6853 2800 50  0000 C CNN
 F 1 "Fuse" V 6944 2800 50  0000 C CNN
-F 2 "Fuse:Fuseholder_Blade_Mini_Keystone_3568" V 6980 2800 50  0001 C CNN
+F 2 "footprints:Fuseholder_Keystone_3522-2" V 6980 2800 50  0001 C CNN
 F 3 "~" H 7050 2800 50  0001 C CNN
+F 4 "3522-2" H 7050 2800 50  0001 C CNN "Part Number"
 	1    7050 2800
 	0    1    1    0
@@
 F 0 "F1" H 4938 2546 50  0000 L CNN
 F 1 "Polyfuse" H 4938 2455 50  0000 L CNN
-F 2 "Diode_SMD:D_SMB" H 4900 2300 50  0001 L CNN
-F 3 "~" H 4850 2500 50  0001 C CNN
+F 2 "Fuse:Fuse_1206_3216Metric" H 4900 2300 50  0001 L CNN
+F 3 "https://pl.mouser.com/datasheet/2/643/ds_CP_0zcj_series-1664160.pdf" H 4850 2500 50  0001 C CNN
+F 4 "0ZCJ0020FF2E" H 5200 2650 50  0001 C CNN "Part Number"
 	1    4850 2500
 	-1   0    0    -1

Commit message: PCB Layout Update 3
Parts:
- removed Q11, Q12, Q8, Q9: Q_PMOS_GSD, Package_TO_SOT_SMD:SOT-23, symbol Device:Q_PMOS_GSD
- added Q11, Q12, Q8, Q9: SiSS05DN, Package_SO:Vishay_PowerPAK_1212-8_Single, symbol Transistor_FET:SiSS27DN
Changed lines of the file:
@@
 	5850 3650 5850 3800
-Wire Wire Line
-	6050 3350 6050 3450
-Connection ~ 6050 3350
-Wire Wire Line
-	6050 3350 6350 3350
 Wire Wire Line
 	6050 3650 6050 3800
@@
 	5950 3350 5950 2250
 Connection ~ 5950 3350
-Wire Wire Line
-	5950 3350 6050 3350
 Connection ~ 5950 5150
 Wire Wire Line
@@
 $EndComp
 $Comp
-L Device:Q_PMOS_GSD Q12
-U 1 1 61C586C2
+L Transistor_FET:SiSS27DN Q8
+U 1 1 61EA3DB0
+P 5350 2350
+F 0 "Q8" V 5692 2350 50  0000 C CNN
+F 1 "SiSS05DN" V 5601 2350 50  0000 C CNN
+F 2 "Package_SO:Vishay_PowerPAK_1212-8_Single" H 5550 2275 50  0001 L CIN
+F 3 "https://www.farnell.com/datasheets/2818743.pdf" V 5350 2350 50  0001 L CNN
+F 4 "SISS05DN-T1-GE3" V 5601 2350 50  0001 C CNN "Part Number"
+	1    5350 2350
+	0    -1   -1   0
+$EndComp
+$Comp
+L Transistor_FET:SiSS27DN Q9
+U 1 1 61EA59E3
+P 5350 3450
+F 0 "Q9" V 5692 3450 50  0000 C CNN
+F 1 "SiSS05DN" V 5601 3450 50  0000 C CNN
+F 2 "Package_SO:Vishay_PowerPAK_1212-8_Single" H 5550 3375 50  0001 L CIN
+F 3 "https://www.farnell.com/datasheets/2818743.pdf" V 5350 3450 50  0001 L CNN
+F 4 "SISS05DN-T1-GE3" H 5350 3450 50  0001 C CNN "Part Number"
+	1    5350 3450
+	0    -1   -1   0
+$EndComp
+$Comp
+L Transistor_FET:SiSS27DN Q11
+U 1 1 61EA704A
+P 6550 2350
+F 0 "Q11" V 6892 2350 50  0000 C CNN
+F 1 "SiSS05DN" V 6801 2350 50  0000 C CNN
+F 2 "Package_SO:Vishay_PowerPAK_1212-8_Single" H 6750 2275 50  0001 L CIN
+F 3 "https://www.farnell.com/datasheets/2818743.pdf" V 6550 2350 50  0001 L CNN
+F 4 "SISS05DN-T1-GE3" H 6550 2350 50  0001 C CNN "Part Number"
+	1    6550 2350
+	0    1    -1   0
+$EndComp
+$Comp
+L Transistor_FET:SiSS27DN Q12
+U 1 1 61EA8267
 P 6550 3450
 F 0 "Q12" V 6892 3450 50  0000 C CNN
-F 1 "Q_PMOS_GSD" V 6801 3450 50  0000 C CNN
-F 2 "Package_TO_SOT_SMD:SOT-23" H 6750 3550 50  0001 C CNN
-F 3 "~" H 6550 3450 50  0001 C CNN
+F 1 "SiSS05DN" V 6801 3450 50  0000 C CNN
+F 2 "Package_SO:Vishay_PowerPAK_1212-8_Single" H 6750 3375 50  0001 L CIN
+F 3 "https://www.farnell.com/datasheets/2818743.pdf" V 6550 3450 50  0001 L CNN
+F 4 "SISS05DN-T1-GE3" H 6550 3450 50  0001 C CNN "Part Number"
 	1    6550 3450
 	0    1    -1   0
 $EndComp
-$Comp
-L Device:Q_PMOS_GSD Q9
-U 1 1 61C60292
-P 5350 3450
-F 0 "Q9" V 5692 3450 50  0000 C CNN
-F 1 "Q_PMOS_GSD" V 5601 3450 50  0000 C CNN
-F 2 "Package_TO_SOT_SMD:SOT-23" H 5550 3550 50  0001 C CNN
-F 3 "~" H 5350 3450 50  0001 C CNN
-	1    5350 3450
-	0    -1   -1   0
-$EndComp
-$Comp
-L Device:Q_PMOS_GSD Q8
-U 1 1 61C62B11
-P 5350 2350
-F 0 "Q8" V 5692 2350 50  0000 C CNN
-F 1 "Q_PMOS_GSD" V 5601 2350 50  0000 C CNN
-F 2 "Package_TO_SOT_SMD:SOT-23" H 5550 2450 50  0001 C CNN
-F 3 "~" H 5350 2350 50  0001 C CNN
-	1    5350 2350
-	0    -1   -1   0
-$EndComp
-$Comp
-L Device:Q_PMOS_GSD Q11
-U 1 1 61C645F3
-P 6550 2350
-F 0 "Q11" V 6892 2350 50  0000 C CNN
-F 1 "Q_PMOS_GSD" V 6801 2350 50  0000 C CNN
-F 2 "Package_TO_SOT_SMD:SOT-23" H 6750 2450 50  0001 C CNN
-F 3 "~" H 6550 2350 50  0001 C CNN
-	1    6550 2350
-	0    1    -1   0
-$EndComp
+Wire Wire Line
+	5950 3350 6050 3350
+Wire Wire Line
+	6050 3350 6350 3350
+Connection ~ 6050 3350
+Wire Wire Line
+	6050 3350 6050 3450
 $EndSCHEMATC

Commit message: Power planes added
Parts:
- Q11, Q12, Q8, Q9: symbol Transistor_FET:SiSS27DN -> BMS_LV_2022-rescue:SiSS27DN-Transistor_FET
Changed lines of the file:
@@
 EESchema Schematic File Version 4
-EELAYER 30 0
+LIBS:BMS_LV_2022-cache
+EELAYER 29 0
 EELAYER END
 $Descr A4 11693 8268
@@
 $EndComp
 $Comp
-L Transistor_FET:SiSS27DN Q8
+L BMS_LV_2022-rescue:SiSS27DN-Transistor_FET Q8
 U 1 1 61EA3DB0
 P 5350 2350
+AR Path="/61EA3DB0" Ref="Q8"  Part="1"
+AR Path="/6269845F/61EA3DB0" Ref="Q8"  Part="1"
 F 0 "Q8" V 5692 2350 50  0000 C CNN
 F 1 "SiSS05DN" V 5601 2350 50  0000 C CNN
@@
 $EndComp
 $Comp
-L Transistor_FET:SiSS27DN Q9
+L BMS_LV_2022-rescue:SiSS27DN-Transistor_FET Q9
 U 1 1 61EA59E3
 P 5350 3450
+AR Path="/61EA59E3" Ref="Q9"  Part="1"
+AR Path="/6269845F/61EA59E3" Ref="Q9"  Part="1"
 F 0 "Q9" V 5692 3450 50  0000 C CNN
 F 1 "SiSS05DN" V 5601 3450 50  0000 C CNN
@@
 $EndComp
 $Comp
-L Transistor_FET:SiSS27DN Q11
+L BMS_LV_2022-rescue:SiSS27DN-Transistor_FET Q11
 U 1 1 61EA704A
 P 6550 2350
+AR Path="/61EA704A" Ref="Q11"  Part="1"
+AR Path="/6269845F/61EA704A" Ref="Q11"  Part="1"
 F 0 "Q11" V 6892 2350 50  0000 C CNN
 F 1 "SiSS05DN" V 6801 2350 50  0000 C CNN
@@
 $EndComp
 $Comp
-L Transistor_FET:SiSS27DN Q12
+L BMS_LV_2022-rescue:SiSS27DN-Transistor_FET Q12
 U 1 1 61EA8267
 P 6550 3450
+AR Path="/61EA8267" Ref="Q12"  Part="1"
+AR Path="/6269845F/61EA8267" Ref="Q12"  Part="1"
 F 0 "Q12" V 6892 3450 50  0000 C CNN
 F 1 "SiSS05DN" V 6801 3450 50  0000 C CNN
