File: HARDWARE/BMS_LV_2022/CAN.kicad_sch (KiCad schematic)
At the start: 9 parts, among them U4 ATA6561-GAQW-N

Commit message: Significant changes
-main connector changed to the other side of the pcb because of using socket connector in the new version
-changed usb mini to usb-c
-changed fuse to 2 fuses protecting current path pins separately
-some minor changes in layout
Parts:
- JP2: footprint Connector_PinHeader_2.54mm:PinHeader_1x02_P2.54mm_Vertical -> Jumper:SolderJumper-2_P1.3mm_Open_TrianglePad1.0x1.5mm
Connections:
- net CANH renamed CAN+
- net CANL renamed CAN-
Changed lines of the file:
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@@
 		)
 	)
-	(hierarchical_label "CANL"
+	(hierarchical_label "CAN-"
 		(shape bidirectional)
 		(at 170.18 102.87 0)
@@
 		)
 	)
-	(hierarchical_label "CANH"
+	(hierarchical_label "CAN+"
 		(shape bidirectional)
 		(at 170.18 97.79 0)
@@
 			)
 		)
-		(property "Footprint" "Connector_PinHeader_2.54mm:PinHeader_1x02_P2.54mm_Vertical"
+		(property "Footprint" "Jumper:SolderJumper-2_P1.3mm_Open_TrianglePad1.0x1.5mm"
 			(at 226.06 95.25 0)
 			(effects
