File: HARDWARE/BMS_LV_2.0-Sandwich/Control-ver2/Thermistors.kicad_sch (KiCad schematic)
At the start: 27 parts, among them J6 Conn_01x09_Female

Commit message: Kolejna kurwa wersja gotowa, japierdole
Parts:
- removed D1: D_Zener_Small, Diode_SMD:D_0805_2012Metric_Pad1.15x1.40mm_HandSolder, symbol Device:D_Zener_Small
- removed R72: 100, Resistor_SMD:R_0603_1608Metric, symbol Device:R_Small
Connections:
- net 3V3_zener renamed 3V3A
Other:
- note removed: "Impedancja wejscia 50K prąd pomiaru gpio 0.5mA dioda zenera wystarczy"
