File: HARDWARE/BMS_LV_2.0-Sandwich/Control-ver2/BMS_LV_2026_Control.kicad_pcb (KiCad board)
At the start: 6 copper layers, 62.5 x 50.9 mm, 80 parts, among them IC1 TAR5S33UTE85LF, IC4 TPS54202HDDCR, J1 Conn_01x26, J3 FTSH-107-01-L-D-K, J6 Conn_01x09_Female, U1 STM32G484RETx, U7 ADM3057ExRW, Y1 ATX-11-F-32.000MHZ-F05-T

Commit message: Druga wersja plytki control skonczona, do review
Parts:
- added D1: D_Zener_Small, Diode_SMD:D_0805_2012Metric_Pad1.15x1.40mm_HandSolder, F.Cu at (151.2, 112.6)
- added R72: 100, Resistor_SMD:R_0603_1608Metric, F.Cu at (149.5, 113.1)
- moved D8 38.2 mm to (144.0, 106.8), turned to 90 degrees
- moved J3 31.6 mm to (151.8, 106.2)
- moved D7 14.5 mm to (162.8, 109.0)
- moved R23 10.3 mm to (165.8, 92.8), turned to -90 degrees
- moved C25 1.62 mm to (148.5, 116.4)
- moved C27 1.62 mm to (151.5, 116.4)
- moved C44 1.62 mm to (154.5, 116.4)
- moved C50 1.62 mm to (157.5, 116.4)
- moved C51 1.62 mm to (160.5, 116.4)
- moved C54 1.62 mm to (163.5, 116.4)
- moved C55 1.62 mm to (166.5, 116.4)
- moved R51 1.62 mm to (147.0, 116.4)
- moved R52 1.62 mm to (150.0, 116.4)
- moved R53 1.62 mm to (153.0, 116.4)
- moved R54 1.62 mm to (156.0, 116.4)
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Connections:
- D7 pad 3: /Control/SWO -> unconnected-(D7-I/O2-Pad3)
- D7 pad 4: /Control/SWCLK -> /Control/SWDIO
- D7 pad 6: /Control/SWDIO -> /Control/SWCLK
- D8 pad 4: /Control/URAT_RX -> /Control/URAT_TX
- D8 pad 6: /Control/URAT_TX -> /Control/URAT_RX
- U1 pad 10: /Therm_8 -> /Therm_6
- U1 pad 17: /Therm_4 -> /Therm_7
- U1 pad 36: /Therm_5 -> /Therm_8
- U1 pad 8: /Therm_6 -> /Therm_4
- U1 pad 9: /Therm_7 -> /Therm_5
Routing:
- net /Control/URAT_TX: track 0.00 -> 105.2 mm, vias 0 -> 1
- net /Control/URAT_RX: track 0.00 -> 97.3 mm, vias 0 -> 1
- net /Control/SWCLK: track 0.00 -> 88.8 mm, vias 0 -> 1
- net /Control/SWDIO: track 0.00 -> 86.0 mm, vias 0 -> 1
- net /Therm_8: track 0.00 -> 80.1 mm, vias 0 -> 1
- net /Therm_7: track 0.00 -> 64.8 mm, vias 0 -> 1
- net /Control/NRST: track 2.32 -> 66.6 mm, vias 0 -> 1
- net /Therm_6: track 0.00 -> 63.4 mm, vias 0 -> 1
- net /Therm_5: track 0.00 -> 62.8 mm, vias 0 -> 1
- net /Therm_4: track 0.00 -> 62.4 mm, vias 0 -> 1
- net /Therm_1: track 0.00 -> 60.9 mm, vias 0 -> 1
- net /Therm_2: track 0.00 -> 60.4 mm, vias 0 -> 1
- net /Therm_3: track 0.00 -> 58.4 mm, vias 0 -> 1
- net /Switch_Signal: track 0.00 -> 55.9 mm, vias 0 -> 4
- net /USB1.USB_DN: track 0.00 -> 54.9 mm, vias 0 -> 1
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- added copper zone on In3.Cu, net /3V3
- added copper zone on In3.Cu, net /5V
- added copper zone on B.Cu, net /CAN/gnd_iso
- added copper zone on F.Cu, net /CAN/gnd_iso
- added copper zone on In1.Cu, net /CAN/gnd_iso
- added copper zone on In2.Cu, net /CAN/gnd_iso
- added copper zone on In3.Cu, net /CAN/gnd_iso
- added copper zone on In4.Cu, net /CAN/gnd_iso
Other:
- board size 62.5 x 50.9 mm -> 62.5 x 45.2 mm

Commit message: Przesunięto złącze do thermistorów oraz programator aby nie bylo kolizji, przesunięto tez bezpieczniki
Parts:
- moved C56 8.52 mm to (178.0, 115.8)
- moved R64 8.52 mm to (176.5, 115.8)
- moved D17 8.01 mm to (156.8, 108.5), turned to 0 degrees
- moved D14 7.22 mm to (156.8, 111.5), turned to 0 degrees
- moved D15 7.01 mm to (156.8, 110.0), turned to 0 degrees
- moved J6 5.53 mm to (152.2, 118.5)
- moved C50 4.09 mm to (153.8, 114.8)
- moved C51 4.09 mm to (156.8, 114.8)
- moved C55 4.09 mm to (162.8, 114.8)
- moved C44 4.08 mm to (150.8, 114.8)
- moved C54 4.08 mm to (159.8, 114.8)
- moved R17 4.00 mm to (160.2, 108.5), turned to 180 degrees
- moved C25 3.75 mm to (144.8, 116.5)
- moved C27 3.75 mm to (147.8, 116.5)
- moved R72 2.39 mm to (149.8, 110.8)
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Connections:
- R72 pad 1: /Thermistors/5V -> /5V
Routing:
- net /Power/EN: track 44.6 -> 30.1 mm, vias 2 -> 3
- net /Thermistors/3V3_zener: track 31.8 -> 45.9 mm
- net /5V: track 40.4 -> 48.7 mm, vias 6 -> 7
- net /Power/+24V safe: track 22.7 -> 28.9 mm
- net GND: track 72.4 -> 68.4 mm, vias 31 -> 32
- net /Therm_8: track 80.1 -> 82.3 mm
- net /Therm_3: track 58.4 -> 60.0 mm
- net /3V3: track 54.1 -> 52.8 mm
- net /Control/NRST: track 66.6 -> 65.5 mm
- net /Control/SWDIO: track 86.0 -> 87.1 mm
- net /Therm_1: track 60.9 -> 59.9 mm
- net /Therm_2: track 60.4 -> 59.4 mm
- net /Therm_7: track 64.8 -> 64.0 mm
- net /Therm_4: track 62.4 -> 63.2 mm
- net /Therm_5: track 62.8 -> 63.4 mm
Other:
- board size 62.5 x 45.2 mm -> 62.5 x 40.8 mm

Commit message: Kolejna kurwa wersja gotowa, japierdole
Parts:
- removed C33: 100n, Capacitor_SMD:C_0603_1608Metric_Pad1.08x0.95mm_HandSolder
- removed D1: D_Zener_Small, Diode_SMD:D_0805_2012Metric_Pad1.15x1.40mm_HandSolder
- removed R72: 100, Resistor_SMD:R_0603_1608Metric
- added C57: 22u, Capacitor_SMD:C_0805_2012Metric_Pad1.18x1.45mm_HandSolder, F.Cu at (182.9, 97.1)
- added C58: 100n, Capacitor_SMD:C_0603_1608Metric, F.Cu at (186.2, 100.0)
- added C59: 22u, Capacitor_SMD:C_0805_2012Metric_Pad1.18x1.45mm_HandSolder, F.Cu at (189.0, 98.8)
- added C60: 100n, Capacitor_SMD:C_0603_1608Metric_Pad1.08x0.95mm_HandSolder, F.Cu at (160.6, 97.5)
- added C61: 100n, Capacitor_SMD:C_0603_1608Metric_Pad1.08x0.95mm_HandSolder, F.Cu at (159.1, 97.5)
- added F6: SMDH2920B150TF, Fuse:Fuse_2920_7451Metric_Pad2.10x5.45mm_HandSolder, F.Cu at (188.5, 85.5)
- added IC2: TAR5S33UTE85LF, Footprint:SOTFL65P210X75-5N, F.Cu at (186.3, 97.9)
- moved C45 42.9 mm to (188.8, 92.8)
- moved R28 41.7 mm to (143.2, 105.0), turned to 90 degrees
- moved C29 40.3 mm to (144.5, 107.5), turned to 0 degrees
- moved Y1 38.1 mm to (161.2, 108.8)
- moved C53 37.5 mm to (164.5, 107.8), turned to -90 degrees
- moved C31 37.3 mm to (186.5, 95.8), turned to 0 degrees
- moved C46 36.7 mm to (184.0, 93.2), turned to 90 degrees
- moved IC1 35.3 mm to (186.2, 93.2), turned to 90 degrees
- moved F3 34.3 mm to (182.5, 85.5), turned to 90 degrees
- moved C52 34.2 mm to (164.5, 111.2), turned to 90 degrees
- moved U1 32.7 mm to (151.5, 102.5), turned to 90 degrees
- moved C34 32.5 mm to (156.5, 109.5), turned to 90 degrees
- moved R20 29.3 mm to (143.2, 90.4)
- moved C30 27.4 mm to (157.6, 96.6), turned to -90 degrees
- moved R19 26.3 mm to (144.7, 90.4)
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Connections:
- D8 pad 4: /Control/URAT_TX -> /Control/URAT_RX
- D8 pad 6: /Control/URAT_RX -> /Control/URAT_TX
- R25 pad 2: /3V3 -> /3V3A
- R51 pad 1: /Thermistors/3V3_zener -> /3V3A
- R52 pad 1: /Thermistors/3V3_zener -> /3V3A
- R53 pad 1: /Thermistors/3V3_zener -> /3V3A
- R54 pad 1: /Thermistors/3V3_zener -> /3V3A
- R55 pad 1: /Thermistors/3V3_zener -> /3V3A
- R56 pad 1: /Thermistors/3V3_zener -> /3V3A
- R63 pad 1: /Thermistors/3V3_zener -> /3V3A
- R64 pad 1: /Thermistors/3V3_zener -> /3V3A
- U1 pad 29: /3V3 -> /3V3A
Routing:
- net /3V3A: track 0.00 -> 103.8 mm, vias 0 -> 3
- net /Control/URAT_TX: track 105.2 -> 20.8 mm
- net /Control/URAT_RX: track 97.3 -> 17.9 mm
- net /Control/SWDIO: track 87.1 -> 20.8 mm
- net /Control/SWCLK: track 88.6 -> 26.9 mm
- net /Thermistors/3V3_zener: track 45.9 -> 0.00 mm
- net /Therm_1: track 59.9 -> 18.6 mm
- net /Therm_7: track 64.0 -> 22.9 mm
- net /Therm_2: track 59.4 -> 18.6 mm
- net /Therm_3: track 60.0 -> 20.5 mm
- net /Therm_8: track 82.3 -> 43.0 mm
- net /Switch_Signal: track 55.9 -> 19.8 mm, vias 4 -> 2
- net /VoltageFuseMeasure: track 53.4 -> 17.5 mm
- net /Therm_6: track 62.9 -> 28.1 mm
- net /Therm_4: track 63.2 -> 28.4 mm
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