File: HARDWARE/BMS_LV_2.0-Sandwich/Power/BMS_LV_2022.kicad_pcb (KiCad board)
At the start: 4 copper layers, 90 x 45 mm, 102 parts, among them J1 Conn_01x26, J11 Conn_01x07_Female, J2 AS214-97PN, J4 Battery+, J5 Battery-, Q1 BC846, Q10 BSS138, Q12 SIR5607DP-T1-RE3, Q13 SIR5607DP-T1-RE3, Q14 SIR5607DP-T1-RE3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

Commit message: Sync
Changed lines of the file:
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@@
 	)
 	(via
-		(at 150.517903 85.33)
+		(at 150.717903 85.83)
 		(size 0.8)
 		(drill 0.4)
@@
 	)
 	(via
-		(at 152.717903 85.33)
+		(at 152.917903 85.73)
 		(size 0.8)
 		(drill 0.4)
@@
 	)
 	(segment
-		(start 132.312903 111.722904)
+		(start 154.912903 81.73)
+		(end 154.617903 82.025)
+		(width 0.21)
+		(layer "In1.Cu")
+		(net 87)
+	)
+	(segment
+		(start 135.303283 108.732523)
+		(end 134.911287 109.12452)
+		(width 0.21)
+		(layer "In1.Cu")
+		(net 87)
+	)
+	(segment
+		(start 135.762903 99.972904)
+		(end 135.762903 103.186178)
+		(width 0.21)
+		(layer "In1.Cu")
+		(net 87)
+	)
+	(segment
+		(start 135.762903 103.186178)
 		(end 135.762903 108.272904)
 		(width 0.21)
@@
 	)
 	(segment
-		(start 132.312903 118.625)
-		(end 132.312903 111.722904)
+		(start 135.762903 108.272904)
+		(end 135.303283 108.732523)
 		(width 0.21)
 		(layer "In1.Cu")
@@
 	)
 	(segment
-		(start 148.162903 87.572904)
+		(start 150.060807 84.175)
 		(end 148.162903 86.072904)
 		(width 0.21)
@@
 	)
 	(segment
-		(start 135.762903 108.272904)
-		(end 135.762903 99.972904)
+		(start 132.312903 118.625)
+		(end 132.312903 111.722904)
 		(width 0.21)
 		(layer "In1.Cu")
@@
 	)
 	(segment
-		(start 153.360807 84.175)
-		(end 154.617903 82.917904)
+		(start 148.162903 87.572904)
+		(end 135.762903 99.972904)
 		(width 0.21)
 		(layer "In1.Cu")
@@
 	)
 	(segment
-		(start 154.617903 82.025)
-		(end 154.912903 81.73)
+		(start 153.360807 84.175)
+		(end 150.060807 84.175)
 		(width 0.21)
 		(layer "In1.Cu")
@@
 	)
 	(segment
-		(start 150.060807 84.175)
+		(start 154.617903 82.917904)
 		(end 153.360807 84.175)
 		(width 0.21)
@@
 	)
 	(segment
-		(start 154.617903 82.917904)
-		(end 154.617903 82.025)
+		(start 134.911287 109.12452)
+		(end 132.312903 111.722904)
 		(width 0.21)
 		(layer "In1.Cu")
@@
 	)
 	(segment
-		(start 148.162903 86.072904)
-		(end 150.060807 84.175)
+		(start 154.617903 82.025)
+		(end 154.617903 82.917904)
 		(width 0.21)
 		(layer "In1.Cu")
@@
 	)
 	(segment
-		(start 135.762903 99.972904)
+		(start 148.162903 86.072904)
 		(end 148.162903 87.572904)
 		(width 0.21)
@@
 		)
 	)
+	(generated
+		(type tuning_pattern)
+		(name "Tuning Pattern")
+		(layer "In1.Cu")
+		(base_line
+			(pts
+				(xy 135.762903 103.186178) (xy 135.762903 108.272904) (xy 134.911287 109.12452)
+			)
+		)
+		(base_line_coupled
+			(pts
+				(arc
+					(start 135.072903 103.12671)
+					(mid 135.015397 103.282573)
+					(end 134.870784 103.365879)
+				)
+			)
+		)
+		(corner_radius_percent 80)
+		(end
+			(xy 134.911287 109.12452)
+		)
+		(initial_side "right")
+		(last_diff_pair_gap 0.18)
+		(last_netname "/USB1-")
+		(last_status "tuned")
+		(last_track_width 0.21)
+		(last_tuning "-0.0213 mm (tuned)")
+		(max_amplitude 1)
+		(min_amplitude 0.2)
+		(min_spacing 0.6)
+		(origin
+			(xy 135.762903 103.186178)
+		)
+		(override_custom_rules no)
+		(rounded yes)
+		(single_sided no)
+		(target_length 1000000)
+		(target_length_max 1000000)
+		(target_length_min 0)
+		(target_skew 0)
+		(target_skew_max 0.1)
+		(target_skew_min -0.1)
+		(tuning_mode "diff_pair_skew")
+		(members "1bee7f0e-543f-4dee-9018-d0ecc0b3e8f0" "1e7cea86-9d32-4145-8b44-e9b771c71211"
+			"2ea70846-ffde-4656-a089-e7ed595ef445"
+		)
+	)

Commit message: V1.0 ready for release
Parts:
- Po chuj to odutowałeś?: renamed from R40
- moved F4 6.28 mm to (143.7, 99.3)
- moved F3 5.80 mm to (144.2, 93.3)
- moved C23 2.90 mm to (157.0, 93.3)
- moved C24 2.90 mm to (162.4, 93.3)
- moved R44 2.90 mm to (158.6, 93.3)
- moved R69 2.90 mm to (160.6, 93.3)
- moved C22 2.24 mm to (154.8, 93.3)
- moved R39 1.85 mm to (152.8, 93.2), turned to -90 degrees
- moved C15 0.30 mm to (140.2, 104.3)
- moved R13 0.25 mm to (127.2, 119.3)
- moved R14 0.25 mm to (127.2, 120.8)
- moved LTC68101 0.17 mm to (155.1, 102.2)
Routing:
- net /V_Out_Pin_1: track 41.5 -> 20.9 mm, vias 1 -> 5
- net +BATT: track 80.2 -> 65.0 mm, vias 80 -> 78
- net Net-(LTC68101-V+): track 22.3 -> 36.4 mm, vias 2 -> 3
- net /V_Out_Pin_2: track 43.2 -> 29.1 mm, vias 1 -> 6
- net Net-(LTC68101-C6): track 26.3 -> 36.7 mm
- net /CAN+: track 58.2 -> 66.0 mm
- net /CAN-: track 58.2 -> 65.9 mm
- net /USB1-: track 53.9 -> 60.9 mm
- net /USB1+: track 53.9 -> 60.8 mm
- net GND: track 46.6 -> 40.1 mm, vias 192 -> 194
- net VCC: track 54.6 -> 48.7 mm
- net /LTC6810/CellBalance5: track 99.5 -> 95.4 mm
- net /MOSI: track 22.0 -> 25.4 mm
- net /MISO: track 20.5 -> 23.8 mm
- net /LTC6810/CellBalance6: track 111.5 -> 109.2 mm
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- added copper zone on B.Cu, net /V_Out_Pin_1
- added copper zone on F.Cu, net /V_Out_Pin_1
- added copper zone on In1.Cu, net /V_Out_Pin_1
- added copper zone on In2.Cu, net /V_Out_Pin_1
- added copper zone on B.Cu, net /V_Out_Pin_2
- added copper zone on F.Cu, net /V_Out_Pin_2
- added copper zone on In1.Cu, net /V_Out_Pin_2
- added copper zone on In2.Cu, net /V_Out_Pin_2
- removed copper zone on B.Cu, net Net-(F3-Pad1)
Other:
- board text added: "10A per channel"
- board text added: "BMS SANDWICH 2026 By Wiktor Krakowski V1.0"
- board text added: "Ballance indicators CELL6 -> CELL 1"
- board text added: "DANGER! HOT"
- board text added: "Danger! HOT"
- board text added: "LTC POWER"
- board text added: "LTC6810"
- board text added: "MAIN FUSES"
- board text added: "ON/OFF & CURRENT SENSE"
- board text added: "Sandwitch Connector"
- board text removed: "B6,B5,B4,B3,B2,B1"
- board text removed: "BMS SANDWICH 2026 By Wiktor Krakowski V2.0 :P"

Commit message: Kicad 10 sync, some silkscreen changes
Parts:
- added G***: LOGO, footprints:propellar_cat_20x20, B.Cu at (131.0, 117.3)
- added G***: LOGO, footprints:pw_love_30x30, B.Cu at (150.0, 101.3)
- moved R34 4.29 mm to (165.5, 107.1), turned to 45 degrees
- moved D9 3.81 mm to (163.7, 116.1)
- moved Q3 3.81 mm to (163.6, 111.4)
- moved R29 3.81 mm to (163.7, 114.3)
- moved D11 1.47 mm to (164.5, 105.6), turned to 45 degrees
- moved Q4 0.56 mm to (165.3, 99.6)
Routing:
- net /LTC6810/Balance3/Sx: track 9.81 -> 15.0 mm
- net Net-(D8-K): track 66.3 -> 69.3 mm
- net /LTC6810/CellBalance4: track 84.0 -> 86.7 mm
- net /LTC6810/Balance2/Sx: track 13.3 -> 16.0 mm
- net /LTC6810/CellBalance3: track 113.0 -> 115.3 mm
- net /eFuse/Gate: track 44.1 -> 46.2 mm
- net Net-(U5-VIOUT): track 7.96 -> 6.16 mm
- net GND: track 40.1 -> 39.1 mm, vias 194 -> 195
- net /LTC6810/CellBalance2: track 97.7 -> 98.7 mm
- net Net-(LTC68101-A0): track 10.7 -> 9.84 mm
- net VCC: vias 48 -> 54
- net Net-(Q12-S): vias 7 -> 14
- net Net-(LTC68101-V+): vias 3 -> 2
- net /LTC6810/CellBalance5: vias 64 -> 63
Other:
- board text added: "BATT+"
- board text added: "GND"
