File: HARDWARE/BMS_LV_2.0-Sandwich/Control/BMS_LV_2026_Control.kicad_pcb (KiCad board)
At the start: 6 copper layers, 62.5 x 40.8 mm, 97 parts, among them IC1 TAR5S33UTE85LF, IC2 TAR5S33UTE85LF, IC4 TPS54202HDDCR, J1 Conn_01x26, J3 FTSH-107-01-L-D-K, J6 Conn_01x09_Female, U1 STM32G484RETx, U7 ADM3057ExRW, Y1 ATX-11-F-32.000MHZ-F05-T

Commit message: Zmieniono tvs, dodano znowu uart, poprawiono silkscreen, gotowy na release
Parts:
- added D11: SMF3.0, Diode_SMD:D_SOD-123F, B.Cu at (184.5, 94.2)
- added D12: SMF3.0, Diode_SMD:D_SOD-123F, B.Cu at (171.5, 93.5)
- added D13: SMF3.0, Diode_SMD:D_SOD-123F, B.Cu at (176.0, 93.5)
- added D5: SMF3.0, Diode_SMD:D_SOD-123F, B.Cu at (187.7, 101.0)
- added D6: SMF3.0, Diode_SMD:D_SOD-123F, B.Cu at (190.5, 87.5)
- added R27: 100k, Resistor_SMD:R_0603_1608Metric_Pad0.98x0.95mm_HandSolder, B.Cu at (157.0, 95.2)
- added R29: 100, Resistor_SMD:R_0603_1608Metric_Pad0.98x0.95mm_HandSolder, B.Cu at (163.0, 93.0)
- D7, D8: value Quad TVS -> SMF3.0; footprint Footprint:SOT65P210X110-6N -> Diode_SMD:D_SOD-123F
- moved D8 9.05 mm to (188.8, 98.5)
- moved D7 8.31 mm to (167.0, 92.2)
- moved D2 2.75 mm to (190.2, 82.8), turned to 90 degrees
Connections:
- D7 pad 1: unconnected-(D7-I/O1-Pad1) -> /Control/NRST
- D8 pad 1: unconnected-(D8-I/O1-Pad1) -> /Control/SWCLK
- U1 pad 52: unconnected-(U1-PC10-Pad52) -> /Control/URAT_RX
- U1 pad 53: unconnected-(U1-PC11-Pad53) -> /Control/URAT_TX
- U1 pad 7: /Control/NRST -> Net-(U1-PG10)
Routing:
- net /Control/URAT_RX: track 0.00 -> 50.4 mm, vias 0 -> 2
- net /Control/URAT_TX: track 0.00 -> 49.1 mm, vias 0 -> 2
- net /Control/NRST: track 63.6 -> 21.5 mm, vias 2 -> 0
- net Net-(U1-PG10): track 0.00 -> 31.4 mm, vias 0 -> 2
- net /Control/SWO: track 62.3 -> 82.9 mm
- net /3V3: track 104.9 -> 84.8 mm, vias 12 -> 10
- net /Control/SWCLK: track 58.8 -> 67.4 mm
- net GND: track 82.2 -> 75.7 mm
- net /Control/SWDIO: track 61.1 -> 63.1 mm
- net /3V3A: track 134.7 -> 133.6 mm
- net /5V: track 59.5 -> 60.4 mm

Commit message: Gotowe do review
Parts:
- moved R29 0.25 mm to (162.8, 93.0)
